Commit message: add basic shapes macros

File: urdf/basic_shapes.urdf.xacro (robot description, xacro)
@@ -5,20 +5,4 @@
   <!-- basic material -->
   <xacro:include filename="$(find urdf_basic_shapes)/urdf/material.urdf.xacro"/>
-  <!-- <link name="base_link">
-   <visual>
-      <origin xyz="0 0 0" rpy="0 0 0"/>
-      <geometry>
-        <box size="1 1 1"/>
-      </geometry>
-      <material name="grey"/>
-    </visual>
-    <collision>
-      <origin xyz="0 0 0" rpy="0 0 0" />
-      <geometry>
-        <box size="1 1 1" />
-      </geometry>
-    </collision>
-    <xacro:solid_cuboid_inertia m="1" h="1" d="1" w="1"/>
-  </link> -->
   <xacro:macro name="cube" params="name x y z ori rpy rgb m">
     <link name="${name}">
@@ -39,10 +23,39 @@
     </link>
   </xacro:macro>
-  <!-- <joint name="cube_joint" type="fixed">
-    <parent link="base_link"/>
-    <child link="cube1"/>
-    <axis xyz="0 0 0"/>
-    <origin xyz="0 0 0" />
-  </joint> -->
-  <xacro:cube name="base_link" x="1" y="1" z="1" ori="0 0 0" rpy="0 0 0" rgb="green" m="1"/>
+  <xacro:macro name="ball" params="name r ori rpy rgb m">
+    <link name="${name}">
+        <visual>
+          <origin xyz="${ori}" rpy="${rpy}"/>
+          <geometry>
+              <sphere radius="${r}"/>
+          </geometry>
+          <material name="${rgb}"/>
+        </visual>
+        <collision>
+        <origin xyz="${ori}" rpy="${rpy}" />
+        <geometry>
+            <sphere radius="${r}" />
+        </geometry>
+        </collision>
+        <xacro:solid_sphere_inertia m="${m}" r="${r}"/>
+    </link>
+  </xacro:macro>
+  <xacro:macro name="cylinder_shape" params="name r h ori rpy rgb m">
+    <link name="${name}">
+        <visual>
+          <origin xyz="${ori}" rpy="${rpy}"/>
+          <geometry>
+              <cylinder radius="${r}" length="${h}"/>
+          </geometry>
+          <material name="${rgb}"/>
+        </visual>
+        <collision>
+        <origin xyz="${ori}" rpy="${rpy}" />
+        <geometry>
+            <cylinder radius="${r}" length="${h}" />
+        </geometry>
+        </collision>
+        <xacro:solid_cylinder_inertia m="${m}" r="${r}" h="${h}"/>
+    </link>
+  </xacro:macro>
 </robot>

File: urdf/inertia.urdf.xacro (robot description, xacro)
@@ -4,29 +4,41 @@
   <!-- TODO Solid sphere of radius r and mass m-->
   <xacro:macro name="solid_sphere_inertia" params="m r">
+  <inertial>
+      <mass value="${m}" />
     <inertia  ixx="${(2*r*r*m)/5}" ixy = "0" ixz = "0"
               iyy="${(2*r*r*m)/5}" iyz = "0"
               izz="${(2*r*r*m)/5}"
      />
+     </inertial>
   </xacro:macro>
   <!-- TODO Hollow sphere of radius r and mass m-->
-  <xacro:macro name="solid_sphere_inertia" params="m r">
+  <xacro:macro name="hollow_sphere_inertia" params="m r">
+  <inertial>
+      <mass value="${m}" />
     <inertia  ixx="${(2*r*r*m)/3}" ixy = "0" ixz = "0"
               iyy="${(2*r*r*m)/3}" iyz = "0"
               izz="${(2*r*r*m)/3}"
      />
+     </inertial>
   </xacro:macro>
   <!-- TODO Solid ellipsoid of semi-axes a, b, c and mass m-->
   <xacro:macro name="ellipsoid_semi_axes_inertia" params="a b c m r">
+  <inertial>
+      <mass value="${m}" />
     <inertia  ixx="${(m*(b*b+c*c))/5}" ixy = "0" ixz = "0"
               iyy="${(m*(a*a+c*c))/5}" iyz = "0"
               izz="${(m*(a*a+b*b))/5}"
      />
+     </inertial>
   </xacro:macro>
   <!-- TODO Right circular cone with radius r, height h and mass m, about the apex -->
   <xacro:macro name="right_circular_cone_inertia" params="m r h">
+  <inertial>
+      <mass value="${m}" />
     <inertia  ixx="${((3*m*(h*h))/5)+((3*m*(r*r))/20)}" ixy = "0" ixz = "0"
               iyy="${((3*m*(h*h))/5)+((3*m*(r*r))/20)}" iyz = "0"
               izz="${(3*m*(r*r))/10}"
      />
+     </inertial>
   </xacro:macro>
   <!-- TODO Solid cuboid of width w, height h, depth d, and mass m -->
@@ -44,15 +56,21 @@
   <!-- TODO Solid cylinder of radius r, height h and mass m -->
   <xacro:macro name="solid_cylinder_inertia" params="m r h">
+  <inertial>
+      <mass value="${m}" />
     <inertia  ixx="${m*(3*r*r+h*h)/12}" ixy = "0" ixz = "0"
               iyy="${m*(3*r*r+h*h)/12}" iyz = "0"
               izz="${m*r*r/2}"
      />
+     </inertial>
   </xacro:macro>
     <!-- TODO Thick-walled cylindrical tube with open ends, of inner radius r1, outer radius r2, length h and mass m -->
     <xacro:macro name="thick_walled_cylinder_inertia" params="m r1 r2 h">
+    <inertial>
+      <mass value="${m}" />
     <inertia  ixx="${m*((3*(r1*r1+r2*r2))+(h*h))/12}" ixy = "0" ixz = "0"
               iyy="${m*((3*(r1*r1+r2*r2))+(h*h))/12}" iyz = "0"
               izz="${m*(r1*r1+r2*r2)/2}"
      />
+     </inertial>
   </xacro:macro>
 </robot>

Commit message: edit gazebo basics

File: urdf/basic_shapes.urdf.xacro (robot description, xacro)
@@ -5,5 +5,7 @@
   <!-- basic material -->
   <xacro:include filename="$(find urdf_basic_shapes)/urdf/material.urdf.xacro"/>
-  <xacro:macro name="cube" params="name x y z ori rpy rgb m">
+  <!-- basic shapes gazebo-->
+  <xacro:include filename="$(find urdf_basic_shapes)/urdf/basic_shapes.gazebo.xacro"/>
+  <xacro:macro name="cube" params="name x y z ori rpy rgb m friction">
     <link name="${name}">
         <visual>
@@ -22,6 +24,7 @@
         <xacro:solid_cuboid_inertia m="${m}" h="${y}" d="${z}" w="${x}"/>
     </link>
+    <xacro:gazebo_params name="${name}" rgb="${rgb}" friction="${friction}"/>
   </xacro:macro>
-  <xacro:macro name="ball" params="name r ori rpy rgb m">
+  <xacro:macro name="ball" params="name r ori rpy rgb m friction">
     <link name="${name}">
         <visual>
@@ -40,6 +43,7 @@
         <xacro:solid_sphere_inertia m="${m}" r="${r}"/>
     </link>
+    <xacro:gazebo_params name="${name}" rgb="${rgb}" friction="${friction}"/>
   </xacro:macro>
-  <xacro:macro name="cylinder_shape" params="name r h ori rpy rgb m">
+  <xacro:macro name="cylinder_shape" params="name r h ori rpy rgb m friction">
     <link name="${name}">
         <visual>
@@ -58,4 +62,5 @@
         <xacro:solid_cylinder_inertia m="${m}" r="${r}" h="${h}"/>
     </link>
+    <xacro:gazebo_params name="${name}" rgb="${rgb}" friction="${friction}"/>
   </xacro:macro>
 </robot>

File: urdf/material.urdf.xacro (robot description, xacro)
@@ -1,17 +1,17 @@
 <?xml version="1.0"?>
 <robot xmlns:xacro="http://wiki.ros.org/xacro">
-  <material name="green">
+  <material name="Green">
     <color rgba="0 1 0 1"/>
   </material>
-  <material name="blue">
+  <material name="Blue">
     <color rgba="0 0 0.8 1"/>
   </material>
-  <material name="black">
+  <material name="Black">
     <color rgba="0 0 0 1"/>
   </material>
-  <material name="white">
+  <material name="White">
     <color rgba="1 1 1 1"/>
   </material>
-  <material name="grey">
+  <material name="Grey">
     <color rgba="0.8 0.8 0.8 1"/>
   </material>
