Commit message: add diff_wheel macro

File: urdf/basic_shapes.gazebo.xacro (robot description, xacro)
@@ -3,5 +3,4 @@
   <xacro:arg name="laser_visual" default="true"/>
   <xacro:property name="update_rate" value="10" />
-  <xacro:property name="M_PI_2" value="1.57079632679"/>
   <xacro:property name="standard_friction" value="0.2" />
   <xacro:property name="wheel_friction" value="10000.0" />

File: urdf/basic_shapes.urdf.xacro (robot description, xacro)
@@ -7,4 +7,6 @@
   <!-- basic shapes gazebo-->
   <xacro:include filename="$(find urdf_basic_shapes)/urdf/basic_shapes.gazebo.xacro"/>
+  <!-- constants -->
+  <xacro:property name="pi" value="3.1415" />
   <xacro:macro name="cube" params="name x y z ori rpy rgb m friction">
     <link name="${name}">

File: urdf/example.urdf.xacro (robot description, xacro)
@@ -3,12 +3,14 @@
     <!-- basic shapes -->
     <xacro:include filename="$(find urdf_basic_shapes)/urdf/basic_shapes.urdf.xacro"/>
+    <!-- diff_wheel -->
+    <xacro:include filename="$(find urdf_basic_shapes)/urdf/diff_wheel.urdf.xacro"/>
     <link name="base_footprint"/>
-    <xacro:cube name="base_link" x="1" y="1" z="1" ori="0 0 0" rpy="0 0 0" rgb="Green" m="1" friction="${standard_friction}"/>
+    <xacro:cube name="base_link" x="2" y="1" z="1" ori="-.5 0 .5" rpy="0 0 0" rgb="Green" m="1" friction="${standard_friction}"/>
     <joint name="cube1_joint" type="fixed">
         <parent link="base_footprint"/>
         <child link="base_link"/>
-        <origin xyz="0 0 0.5" rpy="0 0 0"/>
+        <origin xyz="0 0 0.2" rpy="0 0 0"/>
     </joint>
-    <xacro:ball name="ball1" r="0.5" ori="0 0 0" rpy="0 0 0" rgb="Blue" m="1"/>
+    <xacro:ball name="ball1" r="0.5" ori="0 0 0" rpy="0 0 0" rgb="Blue" m="1" friction="${standard_friction}"/>
     <joint name="joint_ball1" type="fixed">
         <parent link="base_link"/>
@@ -16,5 +18,5 @@
         <origin xyz="0 0 1" rpy="0 0 0"/>
     </joint>
-    <xacro:cylinder_shape name="cylinder1" r="0.5" h="1" ori="0 0 0" rpy="0 0 0" rgb="Black" m="1"/>
+    <xacro:cylinder_shape name="cylinder1" r="0.5" h="1" ori="0 0 0" rpy="0 0 0" rgb="Black" m="1" friction="${standard_friction}"/>
     <joint name="joint_cylinder1" type="fixed">
         <parent link="base_link"/>
@@ -22,3 +24,4 @@
         <origin xyz="0 0 2" rpy="0 0 3.1416"/>
     </joint>
+    <xacro:diff_wheel wheeldiam="0.4" parent="base_link" wheel_separation="1.2"/>
 </robot>

Commit message: add sensors

File: urdf/basic_shapes.gazebo.xacro (robot description, xacro)
@@ -5,5 +5,5 @@
   <xacro:property name="standard_friction" value="0.2" />
   <xacro:property name="wheel_friction" value="10000.0" />
-  <xacro:property name="caster_friction" value="0.1" />
+  <xacro:property name="sliding_friction" value="0.1" />
     <xacro:macro name="gazebo_params" params="name rgb friction">
         <gazebo reference="${name}">
@@ -11,29 +11,8 @@
             <mu1>${friction}</mu1>
             <mu2>${friction}</mu2>
+            <kp value="10000000.0" />
+            <kd value="1.0" />
         </gazebo>
     </xacro:macro>
-  <gazebo>
-    <plugin name="differential_drive_controller" filename="libgazebo_ros_diff_drive.so">
-      <commandTopic>cmd_vel</commandTopic>
-      <odometryTopic>odom</odometryTopic>
-      <odometryFrame>odom</odometryFrame>
-      <odometrySource>world</odometrySource>
-      <!-- publishOdomTF must be false for robot localization ekf node -->
-      <publishOdomTF>true</publishOdomTF>
-      <robotBaseFrame>base_footprint</robotBaseFrame>
-      <publishWheelTF>false</publishWheelTF>
-      <publishTf>true</publishTf>
-      <publishWheelJointState>true</publishWheelJointState>
-      <legacyMode>false</legacyMode>
-      <updateRate>30</updateRate>
-      <leftJoint>wheel_left_joint</leftJoint>
-      <rightJoint>wheel_right_joint</rightJoint>
-      <wheelSeparation>0.770</wheelSeparation>
-      <wheelDiameter>0.150</wheelDiameter>
-      <wheelAcceleration>1</wheelAcceleration>
-      <wheelTorque>10</wheelTorque>
-      <rosDebugLevel>na</rosDebugLevel>
-    </plugin>
-  </gazebo>
   <!-- Gazebo plugin for ROS Control -->
   <gazebo>

File: urdf/basic_shapes.urdf.xacro (robot description, xacro)
@@ -8,5 +8,6 @@
   <xacro:include filename="$(find urdf_basic_shapes)/urdf/basic_shapes.gazebo.xacro"/>
   <!-- constants -->
-  <xacro:property name="pi" value="3.1415" />
+  <xacro:property name="pi" value="3.14159" />
+  <xacro:property name="update_rate" value="50" />
   <xacro:macro name="cube" params="name x y z ori rpy rgb m friction">
     <link name="${name}">

File: urdf/diff_wheel.urdf.xacro (robot description, xacro)
@@ -1,20 +1,56 @@
 <?xml version="1.0"?>
-<robot name="basic_shapes" xmlns:xacro="http://wiki.ros.org/xacro">
+<robot name="diff_wheel" xmlns:xacro="http://wiki.ros.org/xacro">
     <!-- differential drive macro -->
-    <xacro:macro name="diff_wheel" params=" wheeldiam wheel_separation parent">
-        <xacro:cylinder_shape name="left_wheel" r="${wheeldiam/2}" h="0.1" ori="0 0 0" rpy="0 0 0" rgb="Grey" m="0.1" friction="0.5"/>
+    <xacro:macro name="diff_wheel" params=" wheeldiam wheel_separation parent friction">
+        <xacro:cylinder_shape name="left_wheel" r="${wheeldiam/2}" h="0.1" ori="0 0 0" rpy="0 0 0" rgb="Grey" m="0.1" friction="${friction}"/>
         <joint name="left_wheel_joint" type="continuous">
             <axis xyz="0 0 1" rpy="0 0 0" />
             <parent link="${parent}"/>
             <child link="left_wheel"/>
-            <origin xyz="0 ${-wheel_separation/2} 0" rpy="${pi/2} 0 0"/>
+            <origin xyz="0 ${wheel_separation/2} 0" rpy="${-pi/2} 0 0"/>
         </joint>
-        <xacro:cylinder_shape name="right_wheel" r="${wheeldiam/2}" h="0.1" ori="0 0 0" rpy="0 0 0" rgb="Grey" m="0.1" friction="0.5"/>
+        <xacro:cylinder_shape name="right_wheel" r="${wheeldiam/2}" h="0.1" ori="0 0 0" rpy="0 0 0" rgb="Grey" m="0.1" friction="${friction}"/>
         <joint name="right_wheel_joint" type="continuous">
             <axis xyz="0 0 1" rpy="0 0 0" />
             <parent link="${parent}"/>
             <child link="right_wheel"/>
-            <origin xyz="0 ${wheel_separation/2} 0" rpy="${pi/2} 0 0"/>
+            <origin xyz="0 ${-wheel_separation/2} 0" rpy="${-pi/2} 0 0"/>
         </joint>
+        <gazebo>
+        <plugin name="differential_drive_controller" filename="libgazebo_ros_diff_drive.so">
+            <!-- Plugin update rate in Hz -->
+            <updateRate>${update_rate}</updateRate>
+            <!-- Name of left joint, defaults to `left_joint` -->
+            <leftJoint>left_wheel_joint</leftJoint>
+            <!-- Name of right joint, defaults to `right_joint` -->
+            <rightJoint>right_wheel_joint</rightJoint>
+            <!-- The distance from the center of one wheel to the other, in meters, defaults to 0.34 m -->
+            <wheelSeparation>${wheel_separation}</wheelSeparation>
+            <!-- Diameter of the wheels, in meters, defaults to 0.15 m -->
+            <wheelDiameter>${wheeldiam}</wheelDiameter>
+            <!-- Wheel acceleration, in rad/s^2, defaults to 0.0 rad/s^2 -->
+            <wheelAcceleration>1.0</wheelAcceleration>
+            <!-- Maximum torque which the wheels can produce, in Nm, defaults to 5 Nm -->
+            <wheelTorque>20</wheelTorque>
+            <!-- Topic to receive geometry_msgs/Twist message commands, defaults to `cmd_vel` -->
+            <commandTopic>cmd_vel</commandTopic>
+            <!-- Topic to publish nav_msgs/Odometry messages, defaults to `odom` -->
+            <odometryTopic>odom</odometryTopic>
+            <!-- Odometry frame, defaults to `odom` -->
+            <odometryFrame>odom</odometryFrame>
+            <!-- Robot frame to calculate odometry from, defaults to `base_footprint` -->
+            <robotBaseFrame>base_footprint</robotBaseFrame>
+            <!-- Odometry source, 0 for ENCODER, 1 for WORLD, defaults to WORLD -->
+            <odometrySource>1</odometrySource>
+            <!-- Set to true to publish transforms for the wheel links, defaults to false -->
+            <publishWheelTF>true</publishWheelTF>
+            <!-- Set to true to publish transforms for the odometry, defaults to true -->
+            <publishOdom>true</publishOdom>
+            <!-- Set to true to publish sensor_msgs/JointState on /joint_states for the wheel joints, defaults to false -->
+            <publishWheelJointState>true</publishWheelJointState>
+            <!-- Set to true to swap right and left wheels, defaults to true -->
+            <legacyMode>false</legacyMode>
+        </plugin>
+        </gazebo>
     </xacro:macro>
 </robot>

File: urdf/example.urdf.xacro (robot description, xacro)
@@ -5,6 +5,13 @@
     <!-- diff_wheel -->
     <xacro:include filename="$(find urdf_basic_shapes)/urdf/diff_wheel.urdf.xacro"/>
+    <!-- rplidar -->
+    <xacro:include filename="$(find urdf_basic_shapes)/sensors/rplidar.urdf.xacro"/>
+    <!-- velodyne -->
+    <xacro:include filename="$(find urdf_basic_shapes)/sensors/velodyne.urdf.xacro"/>
+    <!-- hokuyo -->
+    <xacro:include filename="$(find urdf_basic_shapes)/sensors/hokuyo.urdf.xacro"/>
     <link name="base_footprint"/>
-    <xacro:cube name="base_link" x="2" y="1" z="1" ori="-.5 0 .5" rpy="0 0 0" rgb="Green" m="1" friction="${standard_friction}"/>
+    <!-- cubeical base_link -->
+    <xacro:cube name="base_link" x="2" y="1" z="1" ori="-.5 0 .5" rpy="0 0 0" rgb="Green" m="2" friction="${standard_friction}"/>
     <joint name="cube1_joint" type="fixed">
         <parent link="base_footprint"/>
@@ -12,5 +19,6 @@
         <origin xyz="0 0 0.2" rpy="0 0 0"/>
     </joint>
-    <xacro:ball name="ball1" r="0.5" ori="0 0 0" rpy="0 0 0" rgb="Blue" m="1" friction="${standard_friction}"/>
+    <!-- ball  -->
+    <xacro:ball name="ball1" r="0.5" ori="0 0 0" rpy="0 0 0" rgb="Blue" m=".5" friction="${standard_friction}"/>
     <joint name="joint_ball1" type="fixed">
         <parent link="base_link"/>
@@ -18,5 +26,6 @@
         <origin xyz="0 0 1" rpy="0 0 0"/>
     </joint>
-    <xacro:cylinder_shape name="cylinder1" r="0.5" h="1" ori="0 0 0" rpy="0 0 0" rgb="Black" m="1" friction="${standard_friction}"/>
+    <!-- cylinder -->
+    <xacro:cylinder_shape name="cylinder1" r="0.5" h="1" ori="0 0 0" rpy="0 0 0" rgb="Black" m=".5" friction="${standard_friction}"/>
     <joint name="joint_cylinder1" type="fixed">
         <parent link="base_link"/>
@@ -24,4 +33,19 @@
         <origin xyz="0 0 2" rpy="0 0 3.1416"/>
     </joint>
-    <xacro:diff_wheel wheeldiam="0.4" parent="base_link" wheel_separation="1.2"/>
+    <!-- diff drive -->
+    <!-- the parent link should be the center of wheel axis -->
+    <xacro:diff_wheel wheeldiam="0.4" wheel_separation="1.2" parent="base_link" friction="200"/>
+    <!-- caster wheel -->
+    <xacro:ball name="casterwheel" r="0.2" ori="0 0 0" rpy="0 0 0" rgb="Grey" m=".5" friction="${sliding_friction}"/>
+    <joint name="joint_casterwheel" type="fixed">
+        <parent link="base_link"/>
+        <child link="casterwheel"/>
+        <origin xyz="-1 0 0" rpy="0 0 0"/>
+    </joint>
+    <!-- rplidar -->
+    <xacro:rplidar name="rplidar" xyz="-1 0 1.05" rpy="0 0 0" parent="base_link" topic="rplidar/scan"/>
+    <!-- Hokuyo Laser -->
+    <xacro:hokuyo name="hokuyo" xyz="-1 0 2.05" rpy="0 0 0" parent="base_link" topic="hokuyu/scan"/>
+    <!-- Veldoyne Lidar  -->
+    <xacro:velodyne16 name="velodyne" xyz="-1 0 1.5" rpy="0 0 0" parent="base_link"/>
 </robot>

File: urdf/material.urdf.xacro (robot description, xacro)
@@ -1,4 +1,7 @@
 <?xml version="1.0"?>
 <robot xmlns:xacro="http://wiki.ros.org/xacro">
+  <material name="Red">
+    <color rgba="1 0 0 1"/>
+  </material>
   <material name="Green">
     <color rgba="0 1 0 1"/>
@@ -16,3 +19,18 @@
     <color rgba="0.8 0.8 0.8 1"/>
   </material>
+  <material name="Yellow">
+    <color rgba="1 1 0 1"/>
+  </material>
+  <material name="Orange">
+    <color rgba="1 0.5 0 1"/>
+  </material>
+  <material name="Brown">
+    <color rgba="0.6 0.4 0.2 1"/>
+  </material>
+  <material name="Purple">
+    <color rgba="0.5 0 0.5 1"/>
+  </material>
+  <material name="Cyan">
+    <color rgba="0 1 1 1"/>
+  </material>
 </robot>
