Commit message: add example

File: examples/example.urdf.xacro (robot description, xacro)
@@ -35,5 +35,5 @@
     <!-- diff drive -->
     <!-- the parent link should be the center of wheel axis -->
-    <xacro:diff_wheel wheeldiam="0.4" wheel_separation="1.2" parent="base_link" friction="200"/>
+    <xacro:diff_wheel wheeldiam="0.4" wheel_separation="1.2" parent="base_link" friction="200" rgb="Grey" h=".1"/>
     <!-- caster wheel -->
     <xacro:ball name="casterwheel" r="0.2" ori="0 0 0" rpy="0 0 0" rgb="Grey" m=".5" friction="${sliding_friction}"/>
@@ -44,5 +44,5 @@
     </joint>
     <!-- rplidar -->
-    <xacro:rplidar name="rplidar" xyz="-1 0 1.05" rpy="0 0 0" parent="base_link" topic="rplidar/scan"/>
+    <xacro:rplidar name="rplidar" xyz="-1 0 1.02" rpy="0 0 0" parent="base_link" topic="rplidar/scan"/>
     <!-- Hokuyo Laser -->
     <xacro:hokuyo name="hokuyo" xyz="-1 0 2.05" rpy="0 0 0" parent="base_link" topic="hokuyu/scan"/>

File: urdf/diff_wheel.urdf.xacro (robot description, xacro)
@@ -2,6 +2,6 @@
 <robot name="diff_wheel" xmlns:xacro="http://wiki.ros.org/xacro">
     <!-- differential drive macro -->
-    <xacro:macro name="diff_wheel" params=" wheeldiam wheel_separation parent friction">
-        <xacro:cylinder_shape name="left_wheel" r="${wheeldiam/2}" h="0.1" ori="0 0 0" rpy="0 0 0" rgb="Grey" m="0.1" friction="${friction}"/>
+    <xacro:macro name="diff_wheel" params=" wheeldiam h wheel_separation parent friction rgb">
+        <xacro:cylinder_shape name="left_wheel" r="${wheeldiam/2}" h="${h}" ori="0 0 0" rpy="0 0 0" rgb="${rgb}" m="0.1" friction="${friction}"/>
         <joint name="left_wheel_joint" type="continuous">
             <axis xyz="0 0 1" rpy="0 0 0" />
@@ -10,5 +10,5 @@
             <origin xyz="0 ${wheel_separation/2} 0" rpy="${-pi/2} 0 0"/>
         </joint>
-        <xacro:cylinder_shape name="right_wheel" r="${wheeldiam/2}" h="0.1" ori="0 0 0" rpy="0 0 0" rgb="Grey" m="0.1" friction="${friction}"/>
+        <xacro:cylinder_shape name="right_wheel" r="${wheeldiam/2}" h="${h}" ori="0 0 0" rpy="0 0 0" rgb="${rgb}" m="0.1" friction="${friction}"/>
         <joint name="right_wheel_joint" type="continuous">
             <axis xyz="0 0 1" rpy="0 0 0" />
