Commit message: delivery bot is a copy of turtlebot

File: examples/deliverybot.urdf.xacro (robot description, xacro)
@@ -15,10 +15,24 @@
         <origin xyz="0 0 0.08" rpy="0 0 0"/>
     </joint>
-    <!-- ball  -->
+    <!-- cubic screen -->
+    <xacro:cube name="screen" x=".15" y=".3" z=".4" ori=".25 0 1" rpy="0 0 0" rgb="Blue" m="1" friction="${standard_friction}"/>
+    <joint name="screen_joint" type="fixed">
+        <parent link="base_link"/>
+        <child link="screen"/>
+        <origin xyz="0 0 0" rpy="0 0 0"/>
+    </joint>
+    <!-- cubic butt -->
+    <xacro:cube name="butt" x=".4" y=".5" z=".4" ori="0 0 0" rpy="0 0 0" rgb="White" m="1" friction="${standard_friction}"/>
+    <joint name="butt_joint" type="fixed">
+        <parent link="base_link"/>
+        <child link="butt"/>
+        <origin xyz="-.1 0 0.2" rpy="0 0 0"/>
+    </joint>
+    <!-- Head  -->
     <xacro:ball name="head" r="0.3" ori="0 0 0" rpy="0 0 0" rgb="White" m="1" friction="${standard_friction}"/>
     <joint name="joint_head" type="fixed">
         <parent link="base_link"/>
         <child link="head"/>
-        <origin xyz="0 0 1.4" rpy="0 0 0"/>
+        <origin xyz="0 0 1.3" rpy="0 0 0"/>
     </joint>
     <!-- diff drive -->
@@ -26,18 +40,18 @@
     <xacro:diff_wheel wheeldiam="0.16" h=".05" wheel_separation=".6" parent="base_link" friction="200" rgb="Black"/>
     <!-- caster wheel back -->
-    <xacro:ball name="casterwheel_back" r="0.05" ori="0 0 0" rpy="0 0 0" rgb="Black" m=".1" friction="${sliding_friction}"/>
+    <xacro:ball name="casterwheel_back" r="0.08" ori="0 0 0" rpy="0 0 0" rgb="Grey" m=".1" friction="${sliding_friction}"/>
     <joint name="joint_casterwheel_back" type="fixed">
         <parent link="base_link"/>
         <child link="casterwheel_back"/>
-        <origin xyz="-.25 0 -.05" rpy="0 0 0"/>
+        <origin xyz="-.25 0 -.0" rpy="0 0 0"/>
     </joint>
     <!-- caster wheel front -->
-    <xacro:ball name="casterwheel_front" r="0.05" ori="0 0 0" rpy="0 0 0" rgb="Black" m=".1" friction="${sliding_friction}"/>
+    <xacro:ball name="casterwheel_front" r="0.08" ori="0 0 0" rpy="0 0 0" rgb="Grey" m=".1" friction="${sliding_friction}"/>
     <joint name="joint_casterwheel_front" type="fixed">
         <parent link="base_link"/>
         <child link="casterwheel_front"/>
-        <origin xyz=".25 0 -.05" rpy="0 0 0"/>
+        <origin xyz=".25 0 -.0" rpy="0 0 0"/>
     </joint>
     <!-- Hokuyo Laser -->
-    <xacro:hokuyo name="hokuyo" xyz="-1 0 2.05" rpy="0 0 0" parent="base_link" topic="hokuyu/scan"/>
+    <xacro:hokuyo name="hokuyo" xyz=".25 0 .25" rpy="${pi} 0 0" parent="base_link" topic="hokuyu/scan"/>
 </robot>

File: sensors/hokuyo.urdf.xacro (robot description, xacro)
@@ -1,5 +1,5 @@
 <?xml version="1.0"?>
 <robot name="hokuyo" xmlns:xacro="http://wiki.ros.org/xacro">
-    <xacro:macro name="hokuyo" params="name parent xyz rpy topic">
+    <xacro:macro name="hokuyo" params="name parent xyz rpy topic frame_id">
         <link name="${name}">
             <collision>
@@ -31,5 +31,5 @@
             <sensor type="gpu_ray" name="head_hokuyo_sensor">
             <pose>0 0 0 0 0 0</pose>
-            <visualize>false</visualize>
+            <visualize>true</visualize>
             <update_rate>40</update_rate>
             <ray>
@@ -59,5 +59,5 @@
             <plugin name="gazebo_ros_head_hokuyo_controller" filename="libgazebo_ros_gpu_laser.so">
                 <topicName>${topic}</topicName>
-                <frameName>hokuyo_link</frameName>
+                <frameName>${frame_id}</frameName>
             </plugin>
             </sensor>

File: urdf/basic_shapes.gazebo.xacro (robot description, xacro)
@@ -16,9 +16,9 @@
     </xacro:macro>
   <!-- Gazebo plugin for ROS Control -->
-  <gazebo>
+  <!-- <gazebo>
     <plugin name="gazebo_ros_control" filename="libgazebo_ros_control.so">
       <robotNamespace>/</robotNamespace>
     </plugin>
-  </gazebo>
+  </gazebo> -->
   <!-- <gazebo reference="front_lidar">
     <material>Gazebo/FlatBlack</material>

File: urdf/diff_wheel.urdf.xacro (robot description, xacro)
@@ -18,5 +18,5 @@
         </joint>
         <gazebo>
-        <plugin name="differential_drive_controller" filename="libgazebo_ros_diff_drive.so">
+        <plugin name="diff_drive_controller" filename="libgazebo_ros_diff_drive.so">
             <!-- Plugin update rate in Hz -->
             <updateRate>${update_rate}</updateRate>
@@ -42,5 +42,5 @@
             <robotBaseFrame>base_footprint</robotBaseFrame>
             <!-- Odometry source, 0 for ENCODER, 1 for WORLD, defaults to WORLD -->
-            <odometrySource>1</odometrySource>
+            <odometrySource>world</odometrySource>
             <!-- Set to true to publish transforms for the wheel links, defaults to false -->
             <publishWheelTF>true</publishWheelTF>
@@ -51,4 +51,7 @@
             <!-- Set to true to swap right and left wheels, defaults to true -->
             <legacyMode>false</legacyMode>
+            <publishOdomTF>true</publishOdomTF>
+            <publishTf>true</publishTf>
+            <rosDebugLevel>na</rosDebugLevel>
         </plugin>
         </gazebo>

Commit message: create tko robot

File: examples/deliverybot.urdf.xacro (robot description, xacro)
@@ -54,4 +54,4 @@
     </joint>
     <!-- Hokuyo Laser -->
-    <xacro:hokuyo name="hokuyo" xyz=".25 0 .25" rpy="${pi} 0 0" parent="base_link" topic="hokuyu/scan"/>
+    <xacro:hokuyo name="base_scan" xyz=".25 0 .25" rpy="${pi} 0 0" parent="base_link" topic="scan"/>
 </robot>

File: sensors/hokuyo.urdf.xacro (robot description, xacro)
@@ -1,5 +1,5 @@
 <?xml version="1.0"?>
 <robot name="hokuyo" xmlns:xacro="http://wiki.ros.org/xacro">
-    <xacro:macro name="hokuyo" params="name parent xyz rpy topic">
+    <xacro:macro name="hokuyo" params="name parent xyz rpy min max">
         <link name="${name}">
             <collision>
@@ -21,5 +21,5 @@
             </inertial>
         </link>
-        <joint name="hokuyo_joint" type="fixed">
+        <joint name="${name}_joint" type="fixed">
             <axis xyz="0 1 0" />
             <origin xyz="${xyz}" rpy="${rpy}"/>
@@ -38,6 +38,6 @@
                     <samples>720</samples>
                     <resolution>1</resolution>
-                    <min_angle>-1.570796</min_angle>
-                    <max_angle>1.570796</max_angle>
+                    <min_angle>${min}</min_angle>
+                    <max_angle>${max}</max_angle>
                 </horizontal>
                 </scan>
@@ -58,5 +58,5 @@
             </ray>
             <plugin name="gazebo_ros_head_hokuyo_controller" filename="libgazebo_ros_gpu_laser.so">
-                <topicName>${topic}</topicName>
+                <topicName>${name}</topicName>
                 <frameName>${name}</frameName>
             </plugin>

Commit message: before tko_robot branch

File: examples/deliverybot.urdf.xacro (robot description, xacro)
@@ -54,4 +54,4 @@
     </joint>
     <!-- Hokuyo Laser -->
-    <xacro:hokuyo name="base_scan" xyz=".25 0 .25" rpy="${pi} 0 0" parent="base_link" min="${-pi/2}" max="${pi}"/>
+    <xacro:hokuyo name="base_scan" xyz=".25 0 .25" rpy="${pi} 0 0" parent="base_link" min_a="${-pi/2}" max_a="${pi}"/>
 </robot>

File: examples/tko_robot.urdf.xacro (robot description, xacro)
@@ -49,9 +49,9 @@
     </joint>
     <!-- Hokuyo Laser Back-->
-    <xacro:hokuyo name="scan_back" xyz="-1.017 0 0" rpy="${pi} 0 ${pi}" parent="base_link" min="${-pi/2}" max="${pi/2}"/>
+    <xacro:hokuyo name="scan_back" xyz="-1.017 0 0" rpy="${pi} 0 ${pi}" parent="base_link" min_a="${-pi/2}" max_a="${pi/2}"/>
     <!-- Hokuyo Laser Left-->
-    <xacro:hokuyo name="scan_left" xyz=".14 0.39 .077" rpy="0 0 0" parent="base_link" min="${-pi/2}" max="${pi}"/>
+    <xacro:hokuyo name="scan_left" xyz=".14 0.39 .077" rpy="0 0 0" parent="base_link" min_a="${-pi/2}" max_a="${pi}"/>
     <!-- Hokuyo Laser Right-->
-    <xacro:hokuyo name="scan_right" xyz=".14 -0.39 .162" rpy="0 0 0" parent="base_link" min="${-pi}" max="${pi/2}"/>
+    <xacro:hokuyo name="scan_right" xyz=".14 -0.39 .162" rpy="0 0 0" parent="base_link" min_a="${-pi}" max_a="${pi/2}"/>
     <!-- Veldoyne Lidar  -->
     <xacro:velodyne16 name="velodyne" xyz="0 0 1.392" rpy="0 0 0" parent="base_link"/>

File: sensors/hokuyo.urdf.xacro (robot description, xacro)
@@ -1,5 +1,5 @@
 <?xml version="1.0"?>
 <robot name="hokuyo" xmlns:xacro="http://wiki.ros.org/xacro">
-    <xacro:macro name="hokuyo" params="name parent xyz rpy min max">
+    <xacro:macro name="hokuyo" params="name parent xyz rpy min_a max_a">
         <link name="${name}">
             <collision>
@@ -29,5 +29,5 @@
         <!-- hokuyo -->
         <gazebo reference="${name}">
-            <sensor type="gpu_ray" name="head_hokuyo_sensor">
+            <sensor type="gpu_ray" name="${name}_hokuyo_sensor">
             <pose>0 0 0 0 0 0</pose>
             <visualize>false</visualize>
@@ -38,6 +38,6 @@
                     <samples>720</samples>
                     <resolution>1</resolution>
-                    <min_angle>${min}</min_angle>
-                    <max_angle>${max}</max_angle>
+                    <min_angle>${min_a}</min_angle>
+                    <max_angle>${max_a}</max_angle>
                 </horizontal>
                 </scan>
@@ -57,5 +57,5 @@
                 </noise>
             </ray>
-            <plugin name="gazebo_ros_head_hokuyo_controller" filename="libgazebo_ros_gpu_laser.so">
+            <plugin name="gazebo_ros_${name}_controller" filename="libgazebo_ros_gpu_laser.so">
                 <topicName>${name}</topicName>
                 <frameName>${name}</frameName>

File: urdf/basic_shapes.urdf.xacro (robot description, xacro)
@@ -8,5 +8,5 @@
   <xacro:include filename="$(find urdf_basic_shapes)/urdf/basic_shapes.gazebo.xacro"/>
   <!-- constants -->
-  <xacro:property name="pi" value="3.14159" />
+  <!-- <xacro:property name="pi" value="3.14159" />  is already defined globally-->
   <xacro:property name="update_rate" value="50" />
   <xacro:macro name="cube" params="name x y z ori rpy rgb m friction">

Commit message: add odom topic to diff wheel

File: examples/deliverybot.urdf.xacro (robot description, xacro)
@@ -35,5 +35,5 @@
     <!-- the parent link should be the center of wheel axis -->
     <xacro:include filename="$(find urdf_basic_shapes)/urdf/diff_wheel.urdf.xacro"/>
-    <xacro:diff_wheel wheeldiam="0.16" h=".05" wheel_separation=".6" parent="base_link" friction="200" rgb="Black" odom_topic="robot_pose_ekf/odom_combined"/>
+    <xacro:diff_wheel wheeldiam="0.16" h=".05" wheel_separation=".6" parent="base_link" friction="200" rgb="Black" odom_topic="odom"/>
     <!-- caster wheel back -->
     <xacro:ball name="casterwheel_back" r="0.08" ori="0 0 0" rpy="0 0 0" rgb="Grey" m=".1" friction="${sliding_friction}"/>

File: urdf/diff_wheel.urdf.xacro (robot description, xacro)
@@ -2,5 +2,5 @@
 <robot name="diff_wheel" xmlns:xacro="http://wiki.ros.org/xacro">
     <!-- differential drive macro -->
-    <xacro:macro name="diff_wheel" params=" wheeldiam h wheel_separation parent friction rgb odom_topic">
+    <xacro:macro name="diff_wheel" params=" wheeldiam h wheel_separation parent friction rgb odom_topic:=odom">
         <xacro:cylinder_shape name="left_wheel" r="${wheeldiam/2}" h="${h}" ori="0 0 0" rpy="0 0 0" rgb="${rgb}" m="0.1" friction="${friction}"/>
         <joint name="left_wheel_joint" type="continuous">

Commit message: prepare model for ekf

File: examples/deliverybot.urdf.xacro (robot description, xacro)
@@ -35,5 +35,5 @@
     <!-- the parent link should be the center of wheel axis -->
     <xacro:include filename="$(find urdf_basic_shapes)/urdf/diff_wheel.urdf.xacro"/>
-    <xacro:diff_wheel wheeldiam="0.16" h=".05" wheel_separation=".6" parent="base_link" friction="200" rgb="Black" odom_topic="odom_ekf"/>
+    <xacro:diff_wheel wheeldiam="0.16" h=".05" wheel_separation=".6" parent="base_link" friction="200" rgb="Black" odom_topic="odom" pub_tf="false"/>
     <!-- caster wheel back -->
     <xacro:ball name="casterwheel_back" r="0.08" ori="0 0 0" rpy="0 0 0" rgb="Grey" m=".1" friction="${sliding_friction}"/>

File: urdf/diff_wheel.urdf.xacro (robot description, xacro)
@@ -2,5 +2,5 @@
 <robot name="diff_wheel" xmlns:xacro="http://wiki.ros.org/xacro">
     <!-- differential drive macro -->
-    <xacro:macro name="diff_wheel" params=" wheeldiam h wheel_separation parent friction rgb odom_topic:=odom">
+    <xacro:macro name="diff_wheel" params=" wheeldiam h wheel_separation parent friction rgb odom_topic:=odom pub_tf:=true">
         <xacro:cylinder_shape name="left_wheel" r="${wheeldiam/2}" h="${h}" ori="0 0 0" rpy="0 0 0" rgb="${rgb}" m="0.1" friction="${friction}"/>
         <joint name="left_wheel_joint" type="continuous">
@@ -51,5 +51,5 @@
             <!-- Set to true to swap right and left wheels, defaults to true -->
             <legacyMode>false</legacyMode>
-            <publishOdomTF>true</publishOdomTF>
+            <publishOdomTF>${pub_tf}</publishOdomTF>
             <publishTf>true</publishTf>
             <rosDebugLevel>na</rosDebugLevel>

Commit message: update diff wheel to real dimensions

File: examples/deliverybot.urdf.xacro (robot description, xacro)
@@ -9,5 +9,5 @@
         <parent link="base_footprint"/>
         <child link="base_link"/>
-        <origin xyz="0 0 0.08" rpy="0 0 0"/>
+        <origin xyz="0 0 0.1" rpy="0 0 0"/>
     </joint>
     <!-- cubic screen -->
@@ -35,7 +35,7 @@
     <!-- the parent link should be the center of wheel axis -->
     <xacro:include filename="$(find urdf_basic_shapes)/urdf/diff_wheel.urdf.xacro"/>
-    <xacro:diff_wheel wheeldiam="0.16" h=".05" wheel_separation=".6" parent="base_link" friction="1000" rgb="Black" odom_topic="odom" pub_tf="false"/>
+    <xacro:diff_wheel wheeldiam="0.2" h=".05" wheel_separation=".38" parent="base_link" friction="1000" rgb="Black" odom_topic="odom" pub_tf="false"/>
     <!-- caster wheel back -->
-    <xacro:ball name="casterwheel_back" r="0.08" ori="0 0 0" rpy="0 0 0" rgb="Grey" m=".1" friction="${sliding_friction}"/>
+    <xacro:ball name="casterwheel_back" r="0.1" ori="0 0 0" rpy="0 0 0" rgb="Grey" m=".1" friction="${sliding_friction}"/>
     <joint name="joint_casterwheel_back" type="fixed">
         <parent link="base_link"/>
@@ -44,5 +44,5 @@
     </joint>
     <!-- caster wheel front -->
-    <xacro:ball name="casterwheel_front" r="0.08" ori="0 0 0" rpy="0 0 0" rgb="Grey" m=".1" friction="${sliding_friction}"/>
+    <xacro:ball name="casterwheel_front" r="0.1" ori="0 0 0" rpy="0 0 0" rgb="Grey" m=".1" friction="${sliding_friction}"/>
     <joint name="joint_casterwheel_front" type="fixed">
         <parent link="base_link"/>
