Commit message: sdd back lidar to deliverybot and rotate cameras

File: examples/deliverybot.urdf (robot description, URDF)
Before this commit: robot deliverybot, 15 links, 14 joints
Links:
- removed link scan
- added link back_scan, mass 1e-5; collision box size=0.1 0.1 0.1; visual box size=0.1 0.1 0.1
- added link front_scan, mass 1e-5; collision box size=0.1 0.1 0.1; visual box size=0.1 0.1 0.1
- link butt: geometry collision box size=0.3 0.5 0.4; visual box size=0.3 0.5 0.4
Joints:
- removed joint scan_joint
- added joint back_scan_joint: type fixed, parent base_link, child back_scan, origin xyz=-.25 0 .05 rpy=0 0 0, axis 0 1 0
- added joint front_scan_joint: type fixed, parent base_link, child front_scan, origin xyz=.25 0 .05 rpy=0 3.141592653589793 0, axis 0 1 0
- joint butt_joint: origin xyz=-.1 0 0.2 rpy=0 0 0 -> xyz=0 0 0.2 rpy=0 0 0
- joint cameraL_joint: origin xyz=.19 0.18 .3 rpy=0 -0.7853981633974483 0.7853981633974483 -> xyz=.19 0.18 .3 rpy=0 0 0.7853981633974483
- joint cameraR_joint: origin xyz=.19 -.18 .3 rpy=3.141592653589793 -0.7853981633974483 -0.7853981633974483 -> xyz=.19 -.18 .3 rpy=3.141592653589793 0 -0.7853981633974483

File: examples/deliverybot.urdf.xacro (robot description, xacro)
@@ -19,9 +19,9 @@
     </joint>
     <!-- cubic butt -->
-    <xacro:cube name="butt" x=".4" y=".5" z=".4" ori="0 0 0" rpy="0 0 0" rgb="White" m="1" friction="${standard_friction}"/>
+    <xacro:cube name="butt" x=".3" y=".5" z=".4" ori="0 0 0" rpy="0 0 0" rgb="White" m="1" friction="${standard_friction}"/>
     <joint name="butt_joint" type="fixed">
         <parent link="base_link"/>
         <child link="butt"/>
-        <origin xyz="-.1 0 0.2" rpy="0 0 0"/>
+        <origin xyz="0 0 0.2" rpy="0 0 0"/>
     </joint>
     <!-- Head  -->
@@ -52,5 +52,6 @@
     <!-- Hokuyo Laser -->
     <xacro:include filename="$(find urdf_basic_shapes)/sensors/hokuyo.urdf.xacro"/>
-    <xacro:hokuyo name="scan" xyz=".25 0 .05" rpy="0 ${pi} 0" parent="base_link" min_a="${-pi}" max_a="${pi}"/>
+    <xacro:hokuyo name="front_scan" xyz=".25 0 .05" rpy="0 ${pi} 0" parent="base_link" min_a="${-pi}" max_a="${pi}"/>
+    <xacro:hokuyo name="back_scan" xyz="-.25 0 .05" rpy="0 0 0" parent="base_link" min_a="${-pi}" max_a="${pi}"/>
      <!-- imu -->
     <xacro:include filename="$(find urdf_basic_shapes)/sensors/imu.urdf.xacro"/>
@@ -59,5 +60,5 @@
     <!-- depth_cam -->
     <xacro:include filename="$(find urdf_basic_shapes)/sensors/depth_cam.urdf.xacro"/>
-    <xacro:depth_cam name="cameraL" xyz=".19 0.18 .3" rpy="0 -${pi/4} ${pi/4}" parent="base_link"/>
-    <xacro:depth_cam name="cameraR" xyz=".19 -.18 .3" rpy="${pi} -${pi/4} -${pi/4}" parent="base_link"/>
+    <xacro:depth_cam name="cameraL" xyz=".19 0.18 .3" rpy="0 0 ${pi/4}" parent="base_link"/>
+    <xacro:depth_cam name="cameraR" xyz=".19 -.18 .3" rpy="${pi} 0 -${pi/4}" parent="base_link"/>
 </robot>
