Commit message: add 2d scan to velodyne on tko robot

File: examples/basic_example.urdf.xacro (robot description, xacro)
@@ -5,5 +5,5 @@
     <link name="base_footprint"/>
     <!-- cubeical base_link -->
-    <xacro:cube name="base_link" x="2" y="1" z="1" ori="-.5 0 .5" rpy="0 0 0" rgb="Green" m="2" friction="${standard_friction}"/>
+    <xacro:cube name="base_link" x="2" y="1" z="1" ori="-.5 0 .5" rpy="0 0 0" rgb="Orange" m="2" friction="${standard_friction}"/>
     <joint name="cube1_joint" type="fixed">
         <parent link="base_footprint"/>

File: examples/deliverybot.urdf.xacro (robot description, xacro)
@@ -35,5 +35,5 @@
     <!-- the parent link should be the center of wheel axis -->
     <xacro:include filename="$(find urdf_basic_shapes)/urdf/diff_wheel.urdf.xacro"/>
-    <xacro:diff_wheel wheeldiam="0.16" h=".05" wheel_separation=".6" parent="base_link" friction="200" rgb="Black"/>
+    <xacro:diff_wheel wheeldiam="0.16" h=".05" wheel_separation=".6" parent="base_link" friction="200" rgb="Black" odom_topic="robot_pose_ekf/odom_combined"/>
     <!-- caster wheel back -->
     <xacro:ball name="casterwheel_back" r="0.08" ori="0 0 0" rpy="0 0 0" rgb="Grey" m=".1" friction="${sliding_friction}"/>
@@ -52,7 +52,7 @@
     <!-- Hokuyo Laser -->
     <xacro:include filename="$(find urdf_basic_shapes)/sensors/hokuyo.urdf.xacro"/>
-    <xacro:hokuyo name="base_scan" xyz=".25 0 .25" rpy="${pi} 0 0" parent="base_link" min_a="${-pi}" max_a="${pi}"/>
+    <xacro:hokuyo name="scan_filtered" xyz=".25 0 .25" rpy="${pi} 0 0" parent="base_link" min_a="${-pi/2}" max_a="${pi/2}"/>
      <!-- imu -->
     <xacro:include filename="$(find urdf_basic_shapes)/sensors/imu.urdf.xacro"/>
-    <xacro:imu name="imu" xyz="0 0 .5" rpy="0 0 0" parent="base_link"/>
+    <xacro:imu name="wit/Imu" xyz="0 0 .5" rpy="0 0 0" parent="base_link"/>
 </robot>

File: examples/tko_robot.urdf.xacro (robot description, xacro)
@@ -35,5 +35,5 @@
     <!-- the parent link should be the center of wheel axis -->
     <xacro:include filename="$(find urdf_basic_shapes)/urdf/diff_wheel.urdf.xacro"/>
-    <xacro:diff_wheel wheeldiam="0.14" h=".035" wheel_separation=".78" parent="base_link" friction="2000" rgb="Black"/>
+    <xacro:diff_wheel wheeldiam="0.14" h=".035" wheel_separation=".78" parent="base_link" friction="2000" rgb="Black" odom_topic="odom"/>
     <!-- caster wheel back -->
     <xacro:ball name="casterwheel_back" r="0.04" ori="0 0 0" rpy="0 0 0" rgb="Black" m="1" friction="${sliding_friction}"/>
@@ -53,4 +53,6 @@
     <xacro:include filename="$(find urdf_basic_shapes)/sensors/velodyne.urdf.xacro"/>
     <xacro:velodyne16 name="velodyne" xyz="0 0 1.392" rpy="0 0 0" parent="base_link"/>
+    <!-- add scan topic to velodyne lidar-->
+    <xacro:hokuyo name="velodyne_2d" xyz="0 0 1.392" rpy="0 0 0" parent="base_link" min_a="${-pi}" max_a="${pi}"/>
     <!-- imu -->
     <xacro:include filename="$(find urdf_basic_shapes)/sensors/imu.urdf.xacro"/>

File: urdf/diff_wheel.urdf.xacro (robot description, xacro)
@@ -2,5 +2,5 @@
 <robot name="diff_wheel" xmlns:xacro="http://wiki.ros.org/xacro">
     <!-- differential drive macro -->
-    <xacro:macro name="diff_wheel" params=" wheeldiam h wheel_separation parent friction rgb">
+    <xacro:macro name="diff_wheel" params=" wheeldiam h wheel_separation parent friction rgb odom_topic">
         <xacro:cylinder_shape name="left_wheel" r="${wheeldiam/2}" h="${h}" ori="0 0 0" rpy="0 0 0" rgb="${rgb}" m="0.1" friction="${friction}"/>
         <joint name="left_wheel_joint" type="continuous">
@@ -36,5 +36,5 @@
             <commandTopic>cmd_vel</commandTopic>
             <!-- Topic to publish nav_msgs/Odometry messages, defaults to `odom` -->
-            <odometryTopic>odom</odometryTopic>
+            <odometryTopic>${odom_topic}</odometryTopic>
             <!-- Odometry frame, defaults to `odom` -->
             <odometryFrame>odom</odometryFrame>

Commit message: 2d lidar sensor working

File: examples/basic_example.urdf.xacro (robot description, xacro)
@@ -37,9 +37,9 @@
     </joint>
     <!-- rplidar -->
-    <!-- <xacro:include filename="$(find urdf_basic_shapes)/sensors/rplidar.urdf.xacro"/>
-    <xacro:rplidar name="rplidar" xyz="-1 0 1.02" rpy="0 0 0" parent="base_link" topic="rplidar/scan"/> -->
+    <xacro:include filename="$(find urdf_basic_shapes)/sensors/rplidar.urdf.xacro"/>
+    <xacro:rplidar name="rplidar" xyz="-1 0 1.02" rpy="0 0 0" parent="base_link" topic="rplidar/scan"/>
     <!-- Hokuyo Laser -->
-    <!-- <xacro:include filename="$(find urdf_basic_shapes)/sensors/hokuyo.urdf.xacro"/>
-    <xacro:hokuyo name="hokuyo_scan" xyz="-1 0 2.05" rpy="0 0 0" parent="base_link" min_a="${-pi/2}" max_a="${pi/2}"/> -->
+    <xacro:include filename="$(find urdf_basic_shapes)/sensors/hokuyo.urdf.xacro"/>
+    <xacro:hokuyo name="hokuyo_scan" xyz="-1 0 2.05" rpy="0 0 0" parent="base_link" min_a="${-pi/2}" max_a="${pi/2}"/>
     <!-- Veldoyne Lidar  -->
     <!-- <xacro:include filename="$(find urdf_basic_shapes)/sensors/velodyne.urdf.xacro"/>

File: sensors/hokuyo.urdf.xacro (robot description, xacro)
@@ -12,5 +12,6 @@
             <origin xyz="0 0 0" rpy="0 0 0"/>
             <geometry>
-                <mesh filename="package://urdf_basic_shapes/meshes/hokuyo.dae"/>
+                <box size="0.1 0.1 0.1"/>
+                <!-- <mesh filename="package://urdf_basic_shapes/meshes/hokuyo.dae"/> -->
             </geometry>
             </visual>
@@ -29,36 +30,36 @@
         <!-- hokuyo -->
         <gazebo reference="${name}">
-            <sensor type="gpu_ray" name="${name}_hokuyo_sensor">
-            <pose>0 0 0 0 0 0</pose>
-            <visualize>false</visualize>
-            <update_rate>40</update_rate>
-            <ray>
+            <sensor name="${name}_hokuyo_sensor" type="ray">
+                <always_on>true</always_on>
+                <visualize>true</visualize>
+                <update_rate>5</update_rate>
+                <ray>
                 <scan>
-                <horizontal>
-                    <samples>720</samples>
-                    <resolution>1</resolution>
-                    <min_angle>${min_a}</min_angle>
-                    <max_angle>${max_a}</max_angle>
-                </horizontal>
+                    <horizontal>
+                    <samples>360</samples>
+                    <resolution>1.000000</resolution>
+                    <min_angle>0.000000</min_angle>
+                    <max_angle>6.280000</max_angle>
+                    </horizontal>
                 </scan>
                 <range>
-                <min>0.10</min>
-                <max>30.0</max>
-                <resolution>0.01</resolution>
+                    <min>0.120000</min>
+                    <max>3.5</max>
+                    <resolution>0.015000</resolution>
                 </range>
                 <noise>
-                <type>gaussian</type>
-                <!-- Noise parameters based on published spec for Hokuyo laser
-                    achieving "+-30mm" accuracy at range < 10m.  A mean of 0.0m and
-                    stddev of 0.01m will put 99.7% of samples within 0.03m of the true
-                    reading. -->
-                <mean>0.0</mean>
-                <stddev>0.01</stddev>
+                    <type>gaussian</type>
+                    <mean>0.0</mean>
+                    <stddev>0.01</stddev>
                 </noise>
-            </ray>
-            <plugin name="gazebo_ros_${name}_controller" filename="libgazebo_ros_gpu_laser.so">
+                </ray>
+                <plugin name="gazebo_ros_${name}_controller" filename="libgazebo_ros_ray_sensor.so">
+                <!-- <ros>
+                    <remapping>~/out:=scan</remapping>
+                </ros> -->
                 <topicName>${name}</topicName>
-                <frameName>${name}</frameName>
-            </plugin>
+                <output_type>sensor_msgs/LaserScan</output_type>
+                <frame_name>${name}</frame_name>
+                </plugin>
             </sensor>
         </gazebo>

File: sensors/rplidar.urdf.xacro (robot description, xacro)
@@ -4,7 +4,8 @@
         <link name="${name}">
             <visual>
-            <origin rpy="${pi/2} 0 ${-pi/2-.3}" xyz="-.02 -.05 0"/>
+            <origin rpy="0 0 0" xyz="0 0 0"/>
             <geometry>
-                <mesh filename="package://urdf_basic_shapes/meshes/rplidar.stl" scale=".002 .002 .002"/>
+                <cylinder radius="0.0575" length="0.05"/>
+                <!-- <mesh filename="package://urdf_basic_shapes/meshes/rplidar.stl" scale=".002 .002 .002"/> -->
             </geometry>
             <material name="Grey"/>
@@ -18,36 +19,35 @@
         <!-- rplidar -->
         <gazebo reference="${name}">
-            <sensor type="gpu_ray" name="${name}">
-            <pose>0 0 0 0 0 0</pose>
-            <visualize>false</visualize>
-            <update_rate>40</update_rate>
-            <ray>
+            <sensor name="lidar" type="ray">
+                <always_on>true</always_on>
+                <visualize>true</visualize>
+                <update_rate>5</update_rate>
+                <ray>
                 <scan>
-                <horizontal>
-                    <samples>720</samples>
-                    <resolution>1</resolution>
-                    <min_angle>${-pi}</min_angle>
-                    <max_angle>${pi}</max_angle>
-                </horizontal>
+                    <horizontal>
+                    <samples>360</samples>
+                    <resolution>1.000000</resolution>
+                    <min_angle>0.000000</min_angle>
+                    <max_angle>6.280000</max_angle>
+                    </horizontal>
                 </scan>
                 <range>
-                <min>0.10</min>
-                <max>30.0</max>
-                <resolution>0.01</resolution>
+                    <min>0.120000</min>
+                    <max>3.5</max>
+                    <resolution>0.015000</resolution>
                 </range>
                 <noise>
-                <type>gaussian</type>
-                <!-- Noise parameters based on published spec for Hokuyo laser
-                    achieving "+-30mm" accuracy at range < 10m.  A mean of 0.0m and
-                    stddev of 0.01m will put 99.7% of samples within 0.03m of the true
-                    reading. -->
-                <mean>0.0</mean>
-                <stddev>0.01</stddev>
+                    <type>gaussian</type>
+                    <mean>0.0</mean>
+                    <stddev>0.01</stddev>
                 </noise>
-            </ray>
-            <plugin name="gazebo_ros_head_hokuyo_controller" filename="libgazebo_ros_gpu_laser.so">
-                <topicName>${topic}</topicName>
-                <frameName>laser_link</frameName>
-            </plugin>
+                </ray>
+                <plugin name="scan" filename="libgazebo_ros_ray_sensor.so">
+                <ros>
+                    <remapping>~/out:=scan</remapping>
+                </ros>
+                <output_type>sensor_msgs/LaserScan</output_type>
+                <frame_name>laser_link</frame_name>
+                </plugin>
             </sensor>
         </gazebo>

Commit message: fixed debth cam TODO: change topics same as realsense

File: examples/basic_example.urdf.xacro (robot description, xacro)
@@ -49,5 +49,5 @@
     <xacro:imu name="imu" xyz="0 0 .5" rpy="0 0 0" parent="base_link"/>
     <!-- depth_cam -->
-    <!-- <xacro:include filename="$(find urdf_basic_shapes)/sensors/depth_cam.urdf.xacro"/>
-    <xacro:depth_cam name="camera" xyz="1 0 .5" rpy="0 0 0" parent="base_link"/> -->
+    <xacro:include filename="$(find urdf_basic_shapes)/sensors/depth_cam.urdf.xacro"/>
+    <xacro:depth_cam name="camera" xyz="1 0 .5" rpy="0 0 0" parent="base_link"/>
 </robot>

File: sensors/depth_cam.urdf.xacro (robot description, xacro)
@@ -2,10 +2,10 @@
 <robot name="depth_cam" xmlns:xacro="http://wiki.ros.org/xacro">
     <xacro:macro name="depth_cam" params="name parent xyz rpy">
-    <xacro:property name="r200_cam_rgb_px" value="0.005"/>
+    <!-- <xacro:property name="r200_cam_rgb_px" value="0.005"/>
     <xacro:property name="r200_cam_rgb_py" value="0.018"/>
     <xacro:property name="r200_cam_rgb_pz" value="0.013"/>
-    <xacro:property name="r200_cam_depth_offset" value="0.01"/>
-    <xacro:arg name="camera_visual" default="false"/>
-    <joint name="base_${name}_joint" type="fixed">
+    <xacro:property name="r200_cam_depth_offset" value="0.01"/> -->
+    <!-- <xacro:arg name="camera_visual" default="false"/> -->
+    <!-- <joint name="base_${name}_joint" type="fixed">
       <origin xyz="${xyz}" rpy="${rpy}" />
       <parent link="${parent}"/>
@@ -17,4 +17,5 @@
         <geometry>
         <mesh filename="package://urdf_basic_shapes/meshes/intel_d435.dae" />
+        <box size="0.012 0.132 0.020"/>
         </geometry>
       </visual>
@@ -49,6 +50,6 @@
     <child link="${name}_depth_optical_frame"/>
   </joint>
-  <link name="${name}_depth_optical_frame"/>
-  <gazebo reference="${name}_rgb_frame">
+  <link name="${name}_depth_optical_frame"/> -->
+  <!-- <gazebo reference="${name}_rgb_frame">
     <sensor type="depth" name="realsense_R200">
       <always_on>true</always_on>
@@ -67,5 +68,5 @@
           </clip>
       </camera>
-      <plugin name="${name}_controller" filename="libgazebo_ros_openni_kinect.so">
+      <plugin name="${name}_controller" filename="libgazebo_ros_camera.so">
         <baseline>0.2</baseline>
         <alwaysOn>true</alwaysOn>
@@ -92,4 +93,137 @@
       </plugin>
     </sensor>
+  </gazebo> -->
+<!-- ####################################################### -->
+  <!-- <link name="${name}">
+    <visual>
+      <origin xyz="0 0 0" rpy="0 0 0"/>
+      <geometry>
+        <box size="0.015 0.130 0.022"/>
+      </geometry>
+    </visual>
+    <collision>
+      <origin xyz="0 0 0" rpy="0 0 0"/>
+      <geometry>
+        <box size="0.015 0.130 0.022"/>
+      </geometry>
+    </collision>
+    <inertial>
+      <origin xyz="0 0 0" rpy="0 0 0"/>
+      <mass value="0.035"/>
+      <inertia ixx="0.001"  ixy="0"  ixz="0" iyy="0.001" iyz="0" izz="0.001" />
+    </inertial>
+  </link>
+  <joint name="${name}_joint" type="fixed">
+    <parent link="base_link"/>
+    <child link="${name}"/>
+    <origin xyz="0.215 0 0.05" rpy="0 0 0"/>
+  </joint>
+  <link name="${name}_depth_frame"/>
+  <joint name="${name}_depth_joint" type="fixed">
+    <origin xyz="0 0 0" rpy="${-pi/2} 0 ${-pi/2}"/>
+    <parent link="${name}"/>
+    <child link="${name}_depth_frame"/>
+  </joint>
+  <gazebo reference="${name}">
+    <sensor name="${name}" type="depth">
+      <visualize>true</visualize>
+      <update_rate>30.0</update_rate>
+      <camera name="${name}">
+        <horizontal_fov>1.047198</horizontal_fov>
+        <image>
+          <width>640</width>
+          <height>480</height>
+          <format>R8G8B8</format>
+        </image>
+        <clip>
+          <near>0.05</near>
+          <far>3</far>
+        </clip>
+      </camera>
+      <plugin name="${name}_controller" filename="libgazebo_ros_camera.so">
+        <baseline>0.2</baseline>
+        <alwaysOn>true</alwaysOn>
+        <updateRate>0.0</updateRate>
+        <frame_name>${name}_depth_frame</frame_name>
+        <pointCloudCutoff>0.5</pointCloudCutoff>
+        <pointCloudCutoffMax>3.0</pointCloudCutoffMax>
+        <distortionK1>0</distortionK1>
+        <distortionK2>0</distortionK2>
+        <distortionK3>0</distortionK3>
+        <distortionT1>0</distortionT1>
+        <distortionT2>0</distortionT2>
+        <CxPrime>0</CxPrime>
+        <Cx>0</Cx>
+        <Cy>0</Cy>
+        <focalLength>0</focalLength>
+        <hackBaseline>0</hackBaseline>
+      </plugin>
+    </sensor>
+  </gazebo> -->
+  <link name="${name}">
+    <visual>
+      <origin xyz="${xyz}" rpy="${rpy}"/>
+      <geometry>
+        <box size="0.015 0.130 0.022"/>
+      </geometry>
+    </visual>
+    <collision>
+      <origin xyz="${xyz}" rpy="${rpy}"/>
+      <geometry>
+        <box size="0.015 0.130 0.022"/>
+      </geometry>
+    </collision>
+    <inertial>
+      <origin xyz="${xyz}" rpy="${rpy}"/>
+      <mass value="0.035"/>
+      <inertia ixx="0.001"  ixy="0"  ixz="0" iyy="0.001" iyz="0" izz="0.001" />
+    </inertial>
+  </link>
+  <joint name="${name}_joint" type="fixed">
+    <parent link="base_link"/>
+    <child link="${name}"/>
+    <origin xyz="0.215 0 0.05" rpy="0 0 0"/>
+  </joint>
+  <link name="${name}_depth_frame"/>
+  <joint name="${name}_depth_joint" type="fixed">
+    <origin xyz="0 0 0" rpy="${-pi/2} 0 ${-pi/2}"/>
+    <parent link="${name}"/>
+    <child link="${name}_depth_frame"/>
+  </joint>
+  <gazebo reference="${name}">
+    <sensor name="depth_${name}" type="depth">
+      <visualize>true</visualize>
+      <update_rate>30.0</update_rate>
+      <camera name="${name}">
+        <horizontal_fov>1.047198</horizontal_fov>
+        <image>
+          <width>640</width>
+          <height>480</height>
+          <format>R8G8B8</format>
+        </image>
+        <clip>
+          <near>0.05</near>
+          <far>3</far>
+        </clip>
+      </camera>
+      <plugin name="depth_${name}_controller" filename="libgazebo_ros_camera.so">
+        <baseline>0.2</baseline>
+        <alwaysOn>true</alwaysOn>
+        <updateRate>0.0</updateRate>
+        <frame_name>${name}_depth_frame</frame_name>
+        <pointCloudCutoff>0.5</pointCloudCutoff>
+        <pointCloudCutoffMax>3.0</pointCloudCutoffMax>
+        <distortionK1>0</distortionK1>
+        <distortionK2>0</distortionK2>
+        <distortionK3>0</distortionK3>
+        <distortionT1>0</distortionT1>
+        <distortionT2>0</distortionT2>
+        <CxPrime>0</CxPrime>
+        <Cx>0</Cx>
+        <Cy>0</Cy>
+        <focalLength>0</focalLength>
+        <hackBaseline>0</hackBaseline>
+      </plugin>
+    </sensor>
   </gazebo>
   </xacro:macro>

File: sensors/rplidar.urdf.xacro (robot description, xacro)
@@ -4,5 +4,5 @@
         <link name="${name}">
             <visual>
-            <origin rpy="0 0 0" xyz="0 0 0"/>
+            <origin rpy="0 0 0" xyz="0 0 0.01"/>
             <geometry>
                 <cylinder radius="0.0575" length="0.05"/>
@@ -48,5 +48,5 @@
                 </ros>
                 <output_type>sensor_msgs/LaserScan</output_type>
-                <frame_name>laser_link</frame_name>
+                <frame_name>${name}</frame_name>
                 </plugin>
             </sensor>

Commit message: update hokuyo laser

File: examples/basic_example.urdf.xacro (robot description, xacro)
@@ -41,5 +41,5 @@
     <!-- Hokuyo Laser -->
     <xacro:include filename="$(find urdf_basic_shapes)/sensors/hokuyo.urdf.xacro"/>
-    <xacro:hokuyo name="hokuyo_scan" xyz="-1 0 2.05" rpy="0 0 0" parent="base_link" min_a="${-pi/2}" max_a="${pi/2}"/>
+    <xacro:hokuyo name="hokuyo_scan" xyz="-1 0 2.05" rpy="0 0 0" parent="base_link" min_a="${-pi/2}" max_a="${pi/2}" topic="hokuyo_scan"/>
     <!-- Veldoyne Lidar  -->
     <xacro:include filename="$(find urdf_basic_shapes)/sensors/velodyne.urdf.xacro"/>

File: examples/deliverybot.urdf.xacro (robot description, xacro)
@@ -52,5 +52,5 @@
     <!-- Hokuyo Laser -->
     <xacro:include filename="$(find urdf_basic_shapes)/sensors/hokuyo.urdf.xacro"/>
-    <xacro:hokuyo name="scan" xyz=".25 0 .05" rpy="0 ${pi} 0" parent="base_link" min_a="${-pi}" max_a="${pi}"/>
+    <xacro:hokuyo name="scan" xyz=".25 0 .05" rpy="0 ${pi} 0" parent="base_link" min_a="${-pi}" max_a="${pi}" topic="scan"/>
      <!-- imu -->
     <xacro:include filename="$(find urdf_basic_shapes)/sensors/imu.urdf.xacro"/>

File: examples/tko_robot.urdf.xacro (robot description, xacro)
@@ -45,14 +45,14 @@
     <!-- Hokuyo Laser Back-->
     <xacro:include filename="$(find urdf_basic_shapes)/sensors/hokuyo.urdf.xacro"/>
-    <xacro:hokuyo name="scan_back" xyz="-1.017 0 0" rpy="${pi} 0 ${pi}" parent="base_link" min_a="${-pi/2}" max_a="${pi/2}"/>
+    <xacro:hokuyo name="scan_back" xyz="-1.017 0 0" rpy="${pi} 0 ${pi}" parent="base_link" min_a="${-pi/2}" max_a="${pi/2}" topic="scan_back"/>
     <!-- Hokuyo Laser Left-->
-    <xacro:hokuyo name="scan_left" xyz=".14 0.43 .077" rpy="0 0 0" parent="base_link" min_a="${-pi/2}" max_a="${pi}"/>
+    <xacro:hokuyo name="scan_left" xyz=".14 0.43 .077" rpy="0 0 0" parent="base_link" min_a="${-pi/2}" max_a="${pi}" topic="scan_left"/>
     <!-- Hokuyo Laser Right-->
-    <xacro:hokuyo name="scan_right" xyz=".14 -0.43 .162" rpy="0 0 0" parent="base_link" min_a="${-pi}" max_a="${pi/2}"/>
+    <xacro:hokuyo name="scan_right" xyz=".14 -0.43 .162" rpy="0 0 0" parent="base_link" min_a="${-pi}" max_a="${pi/2}" topic="scan_right"/>
     <!-- Veldoyne Lidar  -->
     <xacro:include filename="$(find urdf_basic_shapes)/sensors/velodyne.urdf.xacro"/>
     <xacro:velodyne16 name="velodyne" xyz="0 0 1.392" rpy="0 0 0" parent="base_link"/>
     <!-- add scan topic to velodyne lidar-->
-    <xacro:hokuyo name="velodyne_2d" xyz="0 0 1.392" rpy="0 0 0" parent="base_link" min_a="${-pi}" max_a="${pi}"/>
+    <xacro:hokuyo name="olei_lidar" xyz="0 0 1.392" rpy="0 0 0" parent="base_link" min_a="${-pi}" max_a="${pi}" topic="scan"/>
     <!-- imu -->
     <xacro:include filename="$(find urdf_basic_shapes)/sensors/imu.urdf.xacro"/>

File: sensors/hokuyo.urdf.xacro (robot description, xacro)
@@ -1,5 +1,5 @@
 <?xml version="1.0"?>
 <robot name="hokuyo" xmlns:xacro="http://wiki.ros.org/xacro">
-    <xacro:macro name="hokuyo" params="name parent xyz rpy min_a max_a">
+    <xacro:macro name="hokuyo" params="name parent xyz rpy min_a max_a topic=scan">
         <link name="${name}">
             <collision>
@@ -58,5 +58,5 @@
             </ray>
             <plugin name="gazebo_ros_${name}_controller" filename="libgazebo_ros_gpu_laser.so">
-                <topicName>${name}</topicName>
+                <topicName>${topic}</topicName>
                 <frameName>${name}</frameName>
             </plugin>
