Commit message: fix velodyne

File: examples/basic_example.urdf.xacro (robot description, xacro)
@@ -43,6 +43,8 @@
     <xacro:hokuyo name="hokuyo_scan" xyz="-1 0 2.05" rpy="0 0 0" parent="base_link" min_a="${-pi/2}" max_a="${pi/2}"/>
     <!-- Veldoyne Lidar  -->
-    <!-- <xacro:include filename="$(find urdf_basic_shapes)/sensors/velodyne.urdf.xacro"/>
-    <xacro:velodyne16 name="velodyne" xyz="-1 0 1.5" rpy="0 0 0" parent="base_link"/> -->
+    <xacro:include filename="$(find urdf_basic_shapes)/sensors/VLP-16.urdf.xacro"/>
+    <xacro:VLP-16 parent="base_link" name="velodyne" topic="velodyne_points" hz="10" samples="440" gpu="false">
+        <origin xyz="-1 0 1.5" rpy="0 0 0" />
+    </xacro:VLP-16>
     <!-- imu -->
     <xacro:include filename="$(find urdf_basic_shapes)/sensors/imu.urdf.xacro"/>

File: examples/tko_robot.urdf.xacro (robot description, xacro)
@@ -41,17 +41,18 @@
         <parent link="base_link"/>
         <child link="casterwheel_back"/>
-        <origin xyz="-.885 0 -.035" rpy="0 0 0"/>
+        <origin xyz="-.885 0 -.03" rpy="0 0 0"/>
     </joint>
     <!-- Hokuyo Laser Back-->
     <xacro:include filename="$(find urdf_basic_shapes)/sensors/hokuyo.urdf.xacro"/>
-    <xacro:hokuyo name="scan_back" xyz="-1.017 0 0" rpy="${pi} 0 ${pi}" parent="base_link" min_a="${-pi/2}" max_a="${pi/2}"/>
+    <xacro:hokuyo name="scan_back" xyz="-1.017 0 0" rpy="${pi} 0 ${pi}" parent="base_link" min_a="${-pi/2}" max_a="${pi/2}" topic="scan_back"/>
     <!-- Hokuyo Laser Left-->
-    <xacro:hokuyo name="scan_left" xyz=".14 0.43 .077" rpy="0 0 0" parent="base_link" min_a="${-pi/2}" max_a="${pi}"/>
+    <xacro:hokuyo name="scan_left" xyz=".14 0.43 .077" rpy="0 0 0" parent="base_link" min_a="${-pi/2}" max_a="${pi}" topic="scan_left"/>
     <!-- Hokuyo Laser Right-->
-    <xacro:hokuyo name="scan_right" xyz=".14 -0.43 .162" rpy="0 0 0" parent="base_link" min_a="${-pi}" max_a="${pi/2}"/>
+    <xacro:hokuyo name="scan_right" xyz=".14 -0.43 .162" rpy="0 0 0" parent="base_link" min_a="${-pi}" max_a="${pi/2}" topic="scan_right"/>
     <!-- Veldoyne Lidar  -->
-    <!-- <xacro:include filename="$(find urdf_basic_shapes)/sensors/velodyne.urdf.xacro"/>
-    <xacro:velodyne16 name="velodyne" xyz="0 0 1.392" rpy="0 0 0" parent="base_link"/> -->
-    <!-- add scan topic to velodyne lidar-->
+    <xacro:include filename="$(find urdf_basic_shapes)/sensors/VLP-16.urdf.xacro"/>
+    <xacro:VLP-16 parent="base_link" name="velodyne" topic="velodyne_points" hz="10" samples="440" gpu="false">
+        <origin xyz="0 0 1.392" rpy="0 0 0" />
+    </xacro:VLP-16>
     <xacro:hokuyo name="velodyne_2d" xyz="0 0 1.392" rpy="0 0 0" parent="base_link" min_a="${-pi}" max_a="${pi}"/>
     <!-- imu -->

File: sensors/hokuyo.urdf.xacro (robot description, xacro)
@@ -1,5 +1,5 @@
 <?xml version="1.0"?>
 <robot name="hokuyo" xmlns:xacro="http://wiki.ros.org/xacro">
-    <xacro:macro name="hokuyo" params="name parent xyz rpy min_a max_a topic">
+    <xacro:macro name="hokuyo" params="name parent xyz rpy min_a max_a topic:=scan">
         <link name="${name}">
             <collision>

File: sensors/velodyne.urdf.xacro (robot description, xacro)
@@ -6,6 +6,6 @@
         <xacro:arg name="organize_cloud" default="false"/>
         <xacro:property name="organize_cloud" value="$(arg organize_cloud)" />
-        <xacro:include filename="$(find velodyne_description)/urdf/VLP-16.urdf.xacro"/>
-        <xacro:VLP-16 parent="${parent}" name="${name}" topic="velodyne_points" organize_cloud="${organize_cloud}" hz="10" samples="440" gpu="${gpu}">
+        <xacro:include filename="$(find urdf_basic_shapes)/sensors/VLP-16.urdf.xacro"/>
+        <xacro:VLP-16 parent="${parent}" name="${name}" topic="velodyne_points" hz="10" samples="440" gpu="${gpu}">
             <origin xyz="${xyz}" rpy="${rpy}" />
         </xacro:VLP-16>

File: urdf/basic_shapes.gazebo.xacro (robot description, xacro)
@@ -18,73 +18,3 @@
         </gazebo>
     </xacro:macro>
-  <!-- Gazebo plugin for ROS Control -->
-  <!-- <gazebo>
-    <plugin name="gazebo_ros_control" filename="libgazebo_ros_control.so">
-      <robotNamespace>/</robotNamespace>
-    </plugin>
-  </gazebo> -->
-  <!-- <gazebo reference="front_lidar">
-    <material>Gazebo/FlatBlack</material>
-    <sensor type="ray" name="lds_lfcd_sensor">
-      <pose>0 0 0 0 0 0</pose>
-      <visualize>false</visualize>
-      <update_rate>5</update_rate>
-      <ray>
-        <scan>
-          <horizontal>
-            <samples>180</samples>
-            <resolution>1</resolution>
-            <min_angle>${-M_PI_2} </min_angle>
-            <max_angle>${M_PI_2}</max_angle>
-          </horizontal>
-        </scan>
-        <range>
-          <min>0.120</min>
-          <max>3.5</max>
-          <resolution>0.015</resolution>
-        </range>
-        <noise>
-          <type>gaussian</type>
-          <mean>0.0</mean>
-          <stddev>0.01</stddev>
-        </noise>
-      </ray>
-      <plugin name="gazebo_ros_lds_lfcd_controller" filename="libgazebo_ros_laser.so">
-        <topicName>scan/front</topicName>
-        <frameName>front_lidar</frameName>
-      </plugin>
-    </sensor>
-  </gazebo>
-  <gazebo reference="back_lidar">
-    <material>Gazebo/FlatBlack</material>
-    <sensor type="ray" name="lds_lfcd_sensor">
-      <pose>0 0 0 0 0 0</pose>
-      <visualize>false</visualize>
-      <update_rate>5</update_rate>
-      <ray>
-        <scan>
-          <horizontal>
-            <samples>180</samples>
-            <resolution>1</resolution>
-            <min_angle>${M_PI_2} </min_angle>
-            <max_angle>${-M_PI_2}</max_angle>
-          </horizontal>
-        </scan>
-        <range>
-          <min>0.120</min>
-          <max>3.5</max>
-          <resolution>0.015</resolution>
-        </range>
-        <noise>
-          <type>gaussian</type>
-          <mean>0.0</mean>
-          <stddev>0.01</stddev>
-        </noise>
-      </ray>
-      <plugin name="gazebo_ros_lds_lfcd_controller" filename="libgazebo_ros_laser.so">
-        <topicName>scan/back</topicName>
-        <frameName>back_lidar</frameName>
-      </plugin>
-    </sensor>
-  </gazebo> -->
 </robot>

Commit message: add sonar remove rplidar

File: examples/basic_example.urdf.xacro (robot description, xacro)
@@ -1,4 +1,5 @@
 <?xml version="1.0"?>
-<robot name="basic_shapes" xmlns:xacro="http://wiki.ros.org/xacro">
+<robot name="basic_shapes"
+    xmlns:xacro="http://wiki.ros.org/xacro">
     <!-- basic shapes -->
     <xacro:include filename="$(find urdf_basic_shapes)/urdf/basic_shapes.urdf.xacro"/>
@@ -36,7 +37,4 @@
         <origin xyz="-1 0 0" rpy="0 0 0"/>
     </joint>
-    <!-- rplidar -->
-    <xacro:include filename="$(find urdf_basic_shapes)/sensors/rplidar.urdf.xacro"/>
-    <xacro:rplidar name="rplidar" xyz="-1 0 1.02" rpy="0 0 0" parent="base_link" topic="rplidar/scan"/>
     <!-- Hokuyo Laser -->
     <xacro:include filename="$(find urdf_basic_shapes)/sensors/hokuyo.urdf.xacro"/>
@@ -51,3 +49,6 @@
     <xacro:include filename="$(find urdf_basic_shapes)/sensors/depth_cam.urdf.xacro"/>
     <xacro:depth_cam name="camera" xyz="1 0 .5" rpy="0 0 0" parent="base_link"/>
+    <!-- Sonar -->
+    <xacro:include filename="$(find urdf_basic_shapes)/sensors/sonar.urdf.xacro"/>
+    <xacro:sonar name="sonar_range" xyz=".75 0 1" rpy="0 0 0" parent="base_link" min_a="${-pi/2}" max_a="${pi/2}" topic="sonar"/>
 </robot>

File: sensors/hokuyo.urdf.xacro (robot description, xacro)
@@ -1,22 +1,23 @@
 <?xml version="1.0"?>
-<robot name="hokuyo" xmlns:xacro="http://wiki.ros.org/xacro">
+<robot name="hokuyo"
+    xmlns:xacro="http://wiki.ros.org/xacro">
     <xacro:macro name="hokuyo" params="name parent xyz rpy min_a max_a topic=scan">
         <link name="${name}">
             <collision>
-            <origin xyz="0 0 0" rpy="0 0 0"/>
-            <geometry>
-            <box size="0.1 0.1 0.1"/>
-            </geometry>
+                <origin xyz="0 0 0" rpy="0 0 0"/>
+                <geometry>
+                    <box size="0.1 0.1 0.1"/>
+                </geometry>
             </collision>
             <visual>
-            <origin xyz="0 0 0" rpy="0 0 0"/>
-            <geometry>
-                <mesh filename="package://urdf_basic_shapes/meshes/hokuyo.dae"/>
-            </geometry>
+                <origin xyz="0 0 0" rpy="0 0 0"/>
+                <geometry>
+                    <mesh filename="package://urdf_basic_shapes/meshes/hokuyo.dae"/>
+                </geometry>
             </visual>
             <inertial>
-            <mass value="1e-5" />
-            <origin xyz="0 0 0" rpy="0 0 0"/>
-            <inertia ixx="1e-6" ixy="0" ixz="0" iyy="1e-6" iyz="0" izz="1e-6" />
+                <mass value="1e-5" />
+                <origin xyz="0 0 0" rpy="0 0 0"/>
+                <inertia ixx="1e-6" ixy="0" ixz="0" iyy="1e-6" iyz="0" izz="1e-6" />
             </inertial>
         </link>
@@ -30,35 +31,35 @@
         <gazebo reference="${name}">
             <sensor type="ray" name="${name}_hokuyo_sensor">
-            <pose>0 0 0 0 0 0</pose>
-            <visualize>false</visualize>
-            <update_rate>10</update_rate>
-            <ray>
-                <scan>
-                <horizontal>
-                    <samples>720</samples>
-                    <resolution>1</resolution>
-                    <min_angle>${min_a}</min_angle>
-                    <max_angle>${max_a}</max_angle>
-                </horizontal>
-                </scan>
-                <range>
-                <min>0.10</min>
-                <max>30.0</max>
-                <resolution>0.01</resolution>
-                </range>
-                <noise>
-                <type>gaussian</type>
-                <!-- Noise parameters based on published spec for Hokuyo laser
+                <pose>0 0 0 0 0 0</pose>
+                <visualize>false</visualize>
+                <update_rate>10</update_rate>
+                <ray>
+                    <scan>
+                        <horizontal>
+                            <samples>720</samples>
+                            <resolution>1</resolution>
+                            <min_angle>${min_a}</min_angle>
+                            <max_angle>${max_a}</max_angle>
+                        </horizontal>
+                    </scan>
+                    <range>
+                        <min>0.10</min>
+                        <max>30.0</max>
+                        <resolution>0.01</resolution>
+                    </range>
+                    <noise>
+                        <type>gaussian</type>
+                        <!-- Noise parameters based on published spec for Hokuyo laser
                     achieving "+-30mm" accuracy at range < 10m.  A mean of 0.0m and
                     stddev of 0.01m will put 99.7% of samples within 0.03m of the true
                     reading. -->
-                <mean>0.0</mean>
-                <stddev>0.01</stddev>
-                </noise>
-            </ray>
-            <plugin name="gazebo_ros_${name}_controller" filename="libgazebo_ros_laser.so">
-                <topicName>${topic}</topicName>
-                <frameName>${name}</frameName>
-            </plugin>
+                        <mean>0.0</mean>
+                        <stddev>0.01</stddev>
+                    </noise>
+                </ray>
+                <plugin name="gazebo_ros_${name}_controller" filename="libgazebo_ros_laser.so">
+                    <topicName>${topic}</topicName>
+                    <frameName>${name}</frameName>
+                </plugin>
             </sensor>
         </gazebo>

Commit message: add sonar and cam to tko

File: examples/basic_example.urdf.xacro (robot description, xacro)
@@ -51,4 +51,4 @@
     <!-- Sonar -->
     <xacro:include filename="$(find urdf_basic_shapes)/sensors/sonar.urdf.xacro"/>
-    <xacro:sonar name="sonar_range" xyz=".75 0 1" rpy="0 0 0" parent="base_link" min_a="${-pi/2}" max_a="${pi/2}" topic="sonar"/>
+    <xacro:sonar name="sonar_range" xyz=".75 0 1" rpy="0 0 0" parent="base_link" topic="sonar"/>
 </robot>

File: examples/tko_robot.urdf.xacro (robot description, xacro)
@@ -61,3 +61,11 @@
     <xacro:include filename="$(find urdf_basic_shapes)/sensors/imu.urdf.xacro"/>
     <xacro:imu name="imu" xyz="0 0 0" rpy="0 0 0" parent="base_link"/>
+    <!-- depth_cam -->
+    <xacro:include filename="$(find urdf_basic_shapes)/sensors/depth_cam.urdf.xacro"/>
+    <xacro:depth_cam name="cameraF" xyz=".1 0 .5" rpy="0 0 0" parent="base_link"/>
+    <xacro:depth_cam name="cameraB" xyz="-.3 0 .5" rpy="0 0 ${pi}" parent="base_link"/>
+    <!-- Sonar -->
+    <xacro:include filename="$(find urdf_basic_shapes)/sensors/sonar.urdf.xacro"/>
+    <xacro:sonar name="sonarR" xyz="-1.1 -.05 .05" rpy="0 0 ${pi + 0.174533}" parent="base_link" topic="sonarR"/>
+    <xacro:sonar name="sonarL" xyz="-1.1 0.05 .05" rpy="0 0 ${pi - 0.174533}" parent="base_link" topic="sonarL"/>
 </robot>

File: sensors/sonar.urdf.xacro (robot description, xacro)
@@ -2,5 +2,5 @@
 <robot name="hokuyo"
     xmlns:xacro="http://wiki.ros.org/xacro">
-    <xacro:macro name="sonar" params="name parent xyz rpy min_a max_a topic=sonar">
+    <xacro:macro name="sonar" params="name parent xyz rpy min_a=-0.14835 max_a=0.14835 topic=sonar">
         <xacro:cube name="${name}" x="0.05" y="0.05" z="0.05" ori="-.025 0 0" rpy="0 0 0" rgb="Red" m="0.02" friction="${standard_friction}"/>
         <joint name="${name}_joint" type="fixed">
@@ -13,5 +13,5 @@
             <sensor type="ray" name="TeraRanger">
                 <pose>0 0 0 0 0 0</pose>
-                <visualize>true</visualize>
+                <visualize>false</visualize>
                 <update_rate>50</update_rate>
                 <ray>
@@ -20,12 +20,12 @@
                             <samples>10</samples>
                             <resolution>1</resolution>
-                            <min_angle>-0.14835</min_angle>
-                            <max_angle>0.14835</max_angle>
+                            <min_angle>${min_a}</min_angle>
+                            <max_angle>${max_a}</max_angle>
                         </horizontal>
                         <vertical>
                             <samples>10</samples>
                             <resolution>1</resolution>
-                            <min_angle>-0.14835</min_angle>
-                            <max_angle>0.14835</max_angle>
+                            <min_angle>${min_a}</min_angle>
+                            <max_angle>${max_a}</max_angle>
                         </vertical>
                     </scan>
@@ -37,5 +37,5 @@
                 </ray>
                 <plugin filename="libgazebo_ros_range.so" name="gazebo_ros_range">
-                    <gaussianNoise>0.005</gaussianNoise>
+                    <gaussianNoise>0.05</gaussianNoise>
                     <alwaysOn>true</alwaysOn>
                     <updateRate>50</updateRate>
