Commit message: can use mesh again with urdf_launch

File: examples/basic_arm.urdf.xacro (robot description, xacro)
@@ -25,5 +25,5 @@
         <child link="arm1"/>
         <axis xyz="0 1 0"/>
-        <limit lower="0"
+        <limit lower="0"/>
         <origin xyz="0 0 0.05" rpy="0 0 0"/>
     </joint>

File: sensors/depth_cam.urdf.xacro (robot description, xacro)
@@ -4,7 +4,8 @@
     <link name="${name}">
       <visual>
-        <origin xyz="0 0 0" rpy="0 0 0"/>
+        <origin xyz="0 0 0" rpy="${pi/2} 0 ${pi/2}"/>
         <geometry>
-          <box size="0.015 0.130 0.022"/>
+          <!-- <box size="0.015 0.130 0.022"/> -->
+          <mesh filename="package://urdf_basic_shapes/meshes/intel_d435.dae"/>
         </geometry>
       </visual>
