Commit message: edit readme

File: examples/tko_robot.urdf.xacro (robot description, xacro)
@@ -51,6 +51,6 @@
     <xacro:hokuyo name="scan_right" xyz=".14 -0.43 .162" rpy="0 0 0" parent="base_link" min_a="${-pi}" max_a="${pi/2}"/>
     <!-- Veldoyne Lidar  -->
-    <xacro:include filename="$(find urdf_basic_shapes)/sensors/velodyne.urdf.xacro"/>
-    <xacro:velodyne16 name="velodyne" xyz="0 0 1.392" rpy="0 0 0" parent="base_link"/>
+    <!-- <xacro:include filename="$(find urdf_basic_shapes)/sensors/velodyne.urdf.xacro"/>
+    <xacro:velodyne16 name="velodyne" xyz="0 0 1.392" rpy="0 0 0" parent="base_link"/> -->
     <!-- add scan topic to velodyne lidar-->
     <xacro:hokuyo name="velodyne_2d" xyz="0 0 1.392" rpy="0 0 0" parent="base_link" min_a="${-pi}" max_a="${pi}"/>

File: sensors/depth_cam.urdf.xacro (robot description, xacro)
@@ -2,229 +2,70 @@
 <robot name="depth_cam" xmlns:xacro="http://wiki.ros.org/xacro">
     <xacro:macro name="depth_cam" params="name parent xyz rpy">
-    <!-- <xacro:property name="r200_cam_rgb_px" value="0.005"/>
-    <xacro:property name="r200_cam_rgb_py" value="0.018"/>
-    <xacro:property name="r200_cam_rgb_pz" value="0.013"/>
-    <xacro:property name="r200_cam_depth_offset" value="0.01"/> -->
-    <!-- <xacro:arg name="camera_visual" default="false"/> -->
-    <!-- <joint name="base_${name}_joint" type="fixed">
-      <origin xyz="${xyz}" rpy="${rpy}" />
-      <parent link="${parent}"/>
-      <child link="${name}_link" />
-    </joint>
-    <link name="${name}_link">
+    <link name="${name}">
       <visual>
-      <origin xyz="0 0 0" rpy="1.57 0 1.57"/>
+        <origin xyz="0 0 0" rpy="0 0 0"/>
         <geometry>
-        <mesh filename="package://urdf_basic_shapes/meshes/intel_d435.dae" />
-        <box size="0.012 0.132 0.020"/>
+          <box size="0.015 0.130 0.022"/>
         </geometry>
       </visual>
       <collision>
-        <origin xyz="0.003 0.065 0.007" rpy="0 0 0"/>
+        <origin xyz="0 0 0 " rpy="0 0 0 "/>
         <geometry>
-          <box size="0.012 0.132 0.020"/>
+          <box size="0.015 0.130 0.022"/>
         </geometry>
       </collision>
+      <inertial>
+        <origin xyz="0 0 0 " rpy="0 0 0 "/>
+        <mass value="0.035"/>
+        <inertia ixx="0.001"  ixy="0"  ixz="0" iyy="0.001" iyz="0" izz="0.001" />
+      </inertial>
     </link>
-  <joint name="${name}_rgb_joint" type="fixed">
-    <origin xyz="${r200_cam_rgb_px} ${r200_cam_rgb_py} ${r200_cam_rgb_pz}" rpy="0 0 0"/>
-    <parent link="${name}_link"/>
-    <child link="${name}_rgb_frame"/>
-  </joint>
-  <link name="${name}_rgb_frame"/>
-  <joint name="${name}_rgb_optical_joint" type="fixed">
-    <origin xyz="0 0 0" rpy="-1.57 0 -1.57"/>
-    <parent link="${name}_rgb_frame"/>
-    <child link="${name}_rgb_optical_frame"/>
-  </joint>
-  <link name="${name}_rgb_optical_frame"/>
-  <joint name="${name}_depth_joint" type="fixed">
-    <origin xyz="${r200_cam_rgb_px} ${r200_cam_rgb_py + r200_cam_depth_offset} ${r200_cam_rgb_pz}" rpy="0 0 0"/>
-    <parent link="${name}_link"/>
-    <child link="${name}_depth_frame"/>
-  </joint>
-  <link name="${name}_depth_frame"/>
-  <joint name="${name}_depth_optical_joint" type="fixed">
-    <origin xyz="0 0 0" rpy="-1.57 0 -1.57"/>
-    <parent link="${name}_depth_frame"/>
-    <child link="${name}_depth_optical_frame"/>
-  </joint>
-  <link name="${name}_depth_optical_frame"/> -->
-  <!-- <gazebo reference="${name}_rgb_frame">
-    <sensor type="depth" name="realsense_R200">
-      <always_on>true</always_on>
-      <visualize>$(arg camera_visual)</visualize>
-      <camera>
-          <horizontal_fov>1.3439</horizontal_fov>
+    <joint name="${name}_joint" type="fixed">
+      <parent link="${parent}"/>
+      <child link="${name}"/>
+      <origin xyz="${xyz}" rpy="${rpy}"/>
+    </joint>
+    <link name="${name}_depth_frame"/>
+    <joint name="${name}_depth_joint" type="fixed">
+      <origin xyz="0 0 0" rpy="${-pi/2} 0 ${-pi/2}"/>
+      <parent link="${name}"/>
+      <child link="${name}_depth_frame"/>
+    </joint>
+    <gazebo reference="${name}">
+      <sensor name="depth_${name}" type="depth">
+        <visualize>true</visualize>
+        <update_rate>30.0</update_rate>
+        <camera name="${name}">
+          <horizontal_fov>1.047198</horizontal_fov>
           <image>
-              <width>1920</width>
-              <height>1080</height>
-              <format>R8G8B8</format>
+            <width>640</width>
+            <height>480</height>
+            <format>R8G8B8</format>
           </image>
-          <depth_camera></depth_camera>
           <clip>
-              <near>0.03</near>
-              <far>100</far>
+            <near>0.05</near>
+            <far>3</far>
           </clip>
-      </camera>
-      <plugin name="${name}_controller" filename="libgazebo_ros_camera.so">
-        <baseline>0.2</baseline>
-        <alwaysOn>true</alwaysOn>
-        <updateRate>30.0</updateRate>
-        <cameraName>${name}</cameraName>
-        <frameName>${name}_rgb_optical_frame</frameName>
-        <imageTopicName>rgb/image_raw</imageTopicName>
-        <depthImageTopicName>depth/image_raw</depthImageTopicName>
-        <pointCloudTopicName>depth/points</pointCloudTopicName>
-        <cameraInfoTopicName>rgb/${name}_info</cameraInfoTopicName>
-        <depthImageCameraInfoTopicName>depth/${name}_info</depthImageCameraInfoTopicName>
-        <pointCloudCutoff>0.4</pointCloudCutoff>
-            <hackBaseline>0.07</hackBaseline>
-            <distortionK1>0.0</distortionK1>
-            <distortionK2>0.0</distortionK2>
-            <distortionK3>0.0</distortionK3>
-            <distortionT1>0.0</distortionT1>
-            <distortionT2>0.0</distortionT2>
-        <CxPrime>0.0</CxPrime>
-        <Cx>0.0</Cx>
-        <Cy>0.0</Cy>
-        <focalLength>0</focalLength>
-        <hackBaseline>0</hackBaseline>
-      </plugin>
-    </sensor>
-  </gazebo> -->
-<!-- ####################################################### -->
-  <!-- <link name="${name}">
-    <visual>
-      <origin xyz="0 0 0" rpy="0 0 0"/>
-      <geometry>
-        <box size="0.015 0.130 0.022"/>
-      </geometry>
-    </visual>
-    <collision>
-      <origin xyz="0 0 0" rpy="0 0 0"/>
-      <geometry>
-        <box size="0.015 0.130 0.022"/>
-      </geometry>
-    </collision>
-    <inertial>
-      <origin xyz="0 0 0" rpy="0 0 0"/>
-      <mass value="0.035"/>
-      <inertia ixx="0.001"  ixy="0"  ixz="0" iyy="0.001" iyz="0" izz="0.001" />
-    </inertial>
-  </link>
-  <joint name="${name}_joint" type="fixed">
-    <parent link="base_link"/>
-    <child link="${name}"/>
-    <origin xyz="0.215 0 0.05" rpy="0 0 0"/>
-  </joint>
-  <link name="${name}_depth_frame"/>
-  <joint name="${name}_depth_joint" type="fixed">
-    <origin xyz="0 0 0" rpy="${-pi/2} 0 ${-pi/2}"/>
-    <parent link="${name}"/>
-    <child link="${name}_depth_frame"/>
-  </joint>
-  <gazebo reference="${name}">
-    <sensor name="${name}" type="depth">
-      <visualize>true</visualize>
-      <update_rate>30.0</update_rate>
-      <camera name="${name}">
-        <horizontal_fov>1.047198</horizontal_fov>
-        <image>
-          <width>640</width>
-          <height>480</height>
-          <format>R8G8B8</format>
-        </image>
-        <clip>
-          <near>0.05</near>
-          <far>3</far>
-        </clip>
-      </camera>
-      <plugin name="${name}_controller" filename="libgazebo_ros_camera.so">
-        <baseline>0.2</baseline>
-        <alwaysOn>true</alwaysOn>
-        <updateRate>0.0</updateRate>
-        <frame_name>${name}_depth_frame</frame_name>
-        <pointCloudCutoff>0.5</pointCloudCutoff>
-        <pointCloudCutoffMax>3.0</pointCloudCutoffMax>
-        <distortionK1>0</distortionK1>
-        <distortionK2>0</distortionK2>
-        <distortionK3>0</distortionK3>
-        <distortionT1>0</distortionT1>
-        <distortionT2>0</distortionT2>
-        <CxPrime>0</CxPrime>
-        <Cx>0</Cx>
-        <Cy>0</Cy>
-        <focalLength>0</focalLength>
-        <hackBaseline>0</hackBaseline>
-      </plugin>
-    </sensor>
-  </gazebo> -->
-  <link name="${name}">
-    <visual>
-      <origin xyz="${xyz}" rpy="${rpy}"/>
-      <geometry>
-        <box size="0.015 0.130 0.022"/>
-      </geometry>
-    </visual>
-    <collision>
-      <origin xyz="${xyz}" rpy="${rpy}"/>
-      <geometry>
-        <box size="0.015 0.130 0.022"/>
-      </geometry>
-    </collision>
-    <inertial>
-      <origin xyz="${xyz}" rpy="${rpy}"/>
-      <mass value="0.035"/>
-      <inertia ixx="0.001"  ixy="0"  ixz="0" iyy="0.001" iyz="0" izz="0.001" />
-    </inertial>
-  </link>
-  <joint name="${name}_joint" type="fixed">
-    <parent link="base_link"/>
-    <child link="${name}"/>
-    <origin xyz="0.215 0 0.05" rpy="0 0 0"/>
-  </joint>
-  <link name="${name}_depth_frame"/>
-  <joint name="${name}_depth_joint" type="fixed">
-    <origin xyz="0 0 0" rpy="${-pi/2} 0 ${-pi/2}"/>
-    <parent link="${name}"/>
-    <child link="${name}_depth_frame"/>
-  </joint>
-  <gazebo reference="${name}">
-    <sensor name="depth_${name}" type="depth">
-      <visualize>true</visualize>
-      <update_rate>30.0</update_rate>
-      <camera name="${name}">
-        <horizontal_fov>1.047198</horizontal_fov>
-        <image>
-          <width>640</width>
-          <height>480</height>
-          <format>R8G8B8</format>
-        </image>
-        <clip>
-          <near>0.05</near>
-          <far>3</far>
-        </clip>
-      </camera>
-      <plugin name="depth_${name}_controller" filename="libgazebo_ros_camera.so">
-        <baseline>0.2</baseline>
-        <alwaysOn>true</alwaysOn>
-        <updateRate>0.0</updateRate>
-        <frame_name>${name}_depth_frame</frame_name>
-        <pointCloudCutoff>0.5</pointCloudCutoff>
-        <pointCloudCutoffMax>3.0</pointCloudCutoffMax>
-        <distortionK1>0</distortionK1>
-        <distortionK2>0</distortionK2>
-        <distortionK3>0</distortionK3>
-        <distortionT1>0</distortionT1>
-        <distortionT2>0</distortionT2>
-        <CxPrime>0</CxPrime>
-        <Cx>0</Cx>
-        <Cy>0</Cy>
-        <focalLength>0</focalLength>
-        <hackBaseline>0</hackBaseline>
-      </plugin>
-    </sensor>
-  </gazebo>
+        </camera>
+        <plugin name="depth_${name}_controller" filename="libgazebo_ros_camera.so">
+          <baseline>0.2</baseline>
+          <alwaysOn>true</alwaysOn>
+          <updateRate>0.0</updateRate>
+          <frame_name>${name}_depth_frame</frame_name>
+          <pointCloudCutoff>0.5</pointCloudCutoff>
+          <pointCloudCutoffMax>3.0</pointCloudCutoffMax>
+          <distortionK1>0</distortionK1>
+          <distortionK2>0</distortionK2>
+          <distortionK3>0</distortionK3>
+          <distortionT1>0</distortionT1>
+          <distortionT2>0</distortionT2>
+          <CxPrime>0</CxPrime>
+          <Cx>0</Cx>
+          <Cy>0</Cy>
+          <focalLength>0</focalLength>
+          <hackBaseline>0</hackBaseline>
+        </plugin>
+      </sensor>
+    </gazebo>
   </xacro:macro>
 </robot>

Commit message: make tko robot flat

File: examples/tko_robot.urdf.xacro (robot description, xacro)
@@ -41,5 +41,5 @@
         <parent link="base_link"/>
         <child link="casterwheel_back"/>
-        <origin xyz="-.885 0 -.035" rpy="0 0 0"/>
+        <origin xyz="-.885 0 -.03" rpy="0 0 0"/>
     </joint>
     <!-- Hokuyo Laser Back-->

Commit message: urdf matches real robot

File: examples/tko_robot.urdf.xacro (robot description, xacro)
@@ -1,4 +1,5 @@
 <?xml version="1.0"?>
-<robot name="deliverybot" xmlns:xacro="http://wiki.ros.org/xacro">
+<robot name="deliverybot"
+    xmlns:xacro="http://wiki.ros.org/xacro">
     <!-- basic shapes -->
     <xacro:include filename="$(find urdf_basic_shapes)/urdf/basic_shapes.urdf.xacro"/>
@@ -35,5 +36,5 @@
     <!-- the parent link should be the center of wheel axis -->
     <xacro:include filename="$(find urdf_basic_shapes)/urdf/diff_wheel.urdf.xacro"/>
-    <xacro:diff_wheel wheeldiam="0.14" h=".035" wheel_separation=".78" parent="base_link" friction="2000" rgb="Black" odom_topic="odom"/>
+    <xacro:diff_wheel wheeldiam="0.14" h=".035" wheel_separation=".78" parent="base_link" friction="2000" rgb="Black" odom_topic="odom" pub_tf="false"/>
     <!-- caster wheel back -->
     <xacro:ball name="casterwheel_back" r="0.04" ori="0 0 0" rpy="0 0 0" rgb="Black" m="1" friction="${sliding_friction}"/>
@@ -41,5 +42,5 @@
         <parent link="base_link"/>
         <child link="casterwheel_back"/>
-        <origin xyz="-.885 0 -.035" rpy="0 0 0"/>
+        <origin xyz="-.885 0 -.03" rpy="0 0 0"/>
     </joint>
     <!-- Hokuyo Laser Back-->
@@ -47,14 +48,16 @@
     <xacro:hokuyo name="scan_back" xyz="-1.017 0 0" rpy="${pi} 0 ${pi}" parent="base_link" min_a="${-pi/2}" max_a="${pi/2}" topic="scan_back"/>
     <!-- Hokuyo Laser Left-->
-    <xacro:hokuyo name="scan_left" xyz=".14 0.43 .077" rpy="0 0 0" parent="base_link" min_a="${-pi/2}" max_a="${pi}" topic="scan_left"/>
+    <xacro:hokuyo name="scan_left" xyz=".14 0.43 .077" rpy="0 0 ${pi/4}" parent="base_link" min_a="${-pi/2}" max_a="${pi}" topic="scan_left"/>
     <!-- Hokuyo Laser Right-->
-    <xacro:hokuyo name="scan_right" xyz=".14 -0.43 .162" rpy="0 0 0" parent="base_link" min_a="${-pi}" max_a="${pi/2}" topic="scan_right"/>
-    <!-- Veldoyne Lidar  -->
+    <xacro:hokuyo name="scan_right" xyz=".14 -0.43 .162" rpy="0 0 -${pi/4}" parent="base_link" min_a="${-pi}" max_a="${pi/2}" topic="scan_right"/>
+    <!-- TOP 3D Olei Lidar  -->
     <xacro:include filename="$(find urdf_basic_shapes)/sensors/velodyne.urdf.xacro"/>
-    <xacro:velodyne16 name="velodyne" xyz="0 0 1.392" rpy="0 0 0" parent="base_link"/>
+    <xacro:velodyne16 name="olei" xyz="0 0 1.392" rpy="0 0 0" parent="base_link"/>
     <!-- add scan topic to velodyne lidar-->
     <xacro:hokuyo name="olei_lidar" xyz="0 0 1.392" rpy="0 0 0" parent="base_link" min_a="${-pi}" max_a="${pi}" topic="scan"/>
+    <!-- VERTICAL 3D Olei Lidar  -->
+    <!-- <xacro:velodyne16 name="olei_vertical" xyz="0.2 0 1" rpy="0 ${pi*1/4} 0" parent="base_link"/> -->
     <!-- imu -->
     <xacro:include filename="$(find urdf_basic_shapes)/sensors/imu.urdf.xacro"/>
-    <xacro:imu name="imu" xyz="0 0 .5" rpy="0 0 0" parent="base_link"/>
+    <xacro:imu name="imu" xyz="0 0 0" rpy="0 0 0" parent="base_link"/>
 </robot>

Commit message: tko using control

File: examples/tko_robot.urdf.xacro (robot description, xacro)
@@ -35,5 +35,5 @@
     <!-- diff drive -->
     <!-- the parent link should be the center of wheel axis -->
-    <xacro:include filename="$(find urdf_basic_shapes)/urdf/diff_wheel.urdf.xacro"/>
+    <xacro:include filename="$(find urdf_basic_shapes)/urdf/diff_wheel_control.urdf.xacro"/>
     <xacro:diff_wheel wheeldiam="0.14" h=".035" wheel_separation=".78" parent="base_link" friction="2000" rgb="Black" odom_topic="odom" pub_tf="false"/>
     <!-- caster wheel back -->

File: urdf/basic_shapes.gazebo.xacro (robot description, xacro)
@@ -1,4 +1,5 @@
 <?xml version="1.0" ?>
-<robot name="basic_shapes" xmlns:xacro="http://www.ros.org/wiki/xacro" >
+<robot name="basic_shapes"
+  xmlns:xacro="http://www.ros.org/wiki/xacro">
   <xacro:arg name="laser_visual" default="true"/>
   <xacro:property name="update_rate" value="10" />
@@ -6,16 +7,16 @@
   <xacro:property name="wheel_friction" value="10000.0" />
   <xacro:property name="sliding_friction" value="0.1" />
-    <xacro:macro name="gazebo_params" params="name rgb friction">
-        <gazebo reference="${name}">
-            <material>Gazebo/${rgb}</material>
-            <mu1>${friction}</mu1>
-            <mu2>${friction}</mu2>
-            <kp>500000.0</kp>
-            <kd>10.0</kd>
-            <minDepth>0.001</minDepth>
-            <maxVel>0.1</maxVel>
-            <fdir1>1 0 0</fdir1>
-        </gazebo>
-    </xacro:macro>
+  <xacro:macro name="gazebo_params" params="name rgb friction">
+    <gazebo reference="${name}">
+      <material>Gazebo/${rgb}</material>
+      <mu1>${friction}</mu1>
+      <mu2>${friction}</mu2>
+      <kp value="10000000.0" />
+      <kd value="1.0" />
+      <minDepth>0.001</minDepth>
+      <maxVel>0.1</maxVel>
+      <fdir1>1 0 0</fdir1>
+    </gazebo>
+  </xacro:macro>
   <!-- Gazebo plugin for ROS Control -->
   <!-- <gazebo>

Commit message: update tko diff drive for real robot

File: examples/tko_robot.urdf.xacro (robot description, xacro)
@@ -36,5 +36,5 @@
     <!-- the parent link should be the center of wheel axis -->
     <xacro:include filename="$(find urdf_basic_shapes)/urdf/diff_wheel_control.urdf.xacro"/>
-    <xacro:diff_wheel wheeldiam="0.14" h=".035" wheel_separation=".78" parent="base_link" friction="2000" rgb="Black" odom_topic="odom" pub_tf="false"/>
+    <xacro:diff_wheel wheeldiam="0.145" h=".035" wheel_separation=".7" parent="base_link" friction="2000" rgb="Black" odom_topic="odom" pub_tf="false"/>
     <!-- caster wheel back -->
     <xacro:ball name="casterwheel_back" r="0.04" ori="0 0 0" rpy="0 0 0" rgb="Black" m="1" friction="${sliding_friction}"/>

File: urdf/diff_wheel_control.urdf.xacro (robot description, xacro)
@@ -6,8 +6,8 @@
         <xacro:cylinder_shape name="left_wheel" r="${wheeldiam/2}" h="${h}" ori="0 0 0" rpy="0 0 0" rgb="${rgb}" m="0.1" friction="${friction}"/>
         <joint name="left_wheel_joint" type="continuous">
-            <axis xyz="0 0 1" rpy="0 0 0" />
+            <axis xyz="0 0 -1" rpy="0 0 0" />
             <parent link="${parent}"/>
             <child link="left_wheel"/>
-            <origin xyz="0 ${wheel_separation/2} 0" rpy="${-pi/2} 0 0"/>
+            <origin xyz="0 ${wheel_separation/2} 0" rpy="${-pi/2} 0 ${pi}"/>
         </joint>
         <transmission name="left_wheel_trans">
