Commit message: first prototype2

File: examples/tko_robot.urdf.xacro (robot description, xacro)
@@ -6,19 +6,39 @@
     <link name="base_footprint"/>
     <!--cubic base_link -->
-    <xacro:cube name="base_link" x=".325" y=".78" z="1.226" ori="-.0975 0 .613" rpy="0 0 0" rgb="Blue" m="10" friction="${standard_friction}"/>
+    <xacro:cube name="base_link" x=".325" y=".66" z="1.350" ori="-.0975 0 .75" rpy="0 0 0" rgb="Blue" m="10" friction="${standard_friction}"/>
     <joint name="base_joint" type="fixed">
         <parent link="base_footprint"/>
         <child link="base_link"/>
+        <origin xyz="0 0 .075" rpy="0 0 0"/>
+    </joint>
+    <!-- cube -->
+    <xacro:cube name="cube" x=".490" y=".66" z=".100" ori="-.0175 0 .780" rpy="0 0 0" rgb="Blue" m="10" friction="${standard_friction}"/>
+    <joint name="cube_joint" type="fixed">
+        <parent link="base_link"/>
+        <child link="cube"/>
         <origin xyz="0 0 0.075" rpy="0 0 0"/>
     </joint>
     <!-- cylinder -->
-    <xacro:cylinder_shape name="cylinder" r="0.025" h=".25" ori="0 0 0" rpy="0 0 0" rgb="Grey" m=".1" friction="${standard_friction}"/>
+    <xacro:cylinder_shape name="cylinder" r="0.025" h=".100" ori="0 0 0" rpy="0 0 0" rgb="Grey" m=".1" friction="${standard_friction}"/>
     <joint name="joint_cylinder" type="fixed">
         <parent link="base_link"/>
         <child link="cylinder"/>
-        <origin xyz="0 0 1.32" rpy="0 0 0"/>
+        <origin xyz="0 0 1.43" rpy="0 0 0"/>
+    </joint>
+    <!-- hands -->
+    <xacro:cube name="handR" x=".6365" y=".095" z=".100" ori="-${.6365/2}  0 0" rpy="0 0 0" rgb="Blue" m="10" friction="${standard_friction}"/>
+    <joint name="handR_joint" type="fixed">
+        <parent link="base_link"/>
+        <child link="handR"/>
+        <origin xyz="-.2475 -.3775 0.585" rpy="0 0 0"/>
+    </joint>
+    <xacro:cube name="handL" x=".6365" y=".095" z=".100" ori="-${.6365/2} 0 0" rpy="0 0 0" rgb="Blue" m="10" friction="${standard_friction}"/>
+    <joint name="handL_joint" type="fixed">
+        <parent link="base_link"/>
+        <child link="handL"/>
+        <origin xyz="-.2475 .3775 0.585" rpy="0 0 0"/>
     </joint>
     <!-- tail -->
-    <xacro:cube name="tail" x="1.065" y=".2" z=".05" ori="-0.5325 0 0" rpy="0 0 0" rgb="Grey" m="3" friction="${standard_friction}"/>
+    <xacro:cube name="tail" x="1.06169" y=".2" z=".05" ori="-${1.06169/2} 0 0" rpy="0 0 0" rgb="Grey" m="3" friction="${standard_friction}"/>
     <joint name="tail_joint" type="fixed">
         <parent link="base_link"/>
@@ -31,5 +51,5 @@
         <parent link="base_link"/>
         <child link="screen"/>
-        <origin xyz="0.0 0.1 1" rpy="0 0 0"/>
+        <origin xyz="0 0 1" rpy="0 0 0"/>
     </joint>
     <!-- diff drive -->
@@ -42,16 +62,16 @@
         <parent link="base_link"/>
         <child link="casterwheel_back"/>
-        <origin xyz="-.885 0 -.03" rpy="0 0 0"/>
+        <origin xyz="-.884 0 -.03" rpy="0 0 0"/>
     </joint>
     <!-- Hokuyo Laser Back-->
     <xacro:include filename="$(find urdf_basic_shapes)/sensors/hokuyo.urdf.xacro"/>
-    <xacro:hokuyo name="scan_back" xyz="-1.017 0 0" rpy="${pi} 0 ${pi}" parent="base_link" min_a="${-pi/2}" max_a="${pi/2}" topic="/lidarBack/scan"/>
+    <xacro:hokuyo name="scan_back" xyz="-.9765 0 0" rpy="${pi} 0 ${pi}" parent="base_link" min_a="${-pi/2}" max_a="${pi/2}" topic="/lidarBack/scan"/>
     <!-- Hokuyo Laser Front-->
     <xacro:hokuyo name="scan_front" xyz=".14 0.0 .077" rpy="0 0 0" parent="base_link" min_a="${-pi/2}" max_a="${pi/2}" topic="/lidarFront/scan"/>
     <!-- TOP 3D Olei Lidar  -->
     <xacro:include filename="$(find urdf_basic_shapes)/sensors/velodyne.urdf.xacro"/>
-    <xacro:velodyne16 name="olei" xyz="0 0 1.392" rpy="0 0 0" parent="base_link"/>
+    <xacro:velodyne16 name="olei" xyz="0 0 1.515" rpy="0 0 0" parent="base_link"/>
     <!-- add scan topic to velodyne lidar-->
-    <xacro:hokuyo name="olei_lidar" xyz="0 0 1.392" rpy="0 0 0" parent="base_link" min_a="${-pi}" max_a="${pi}" topic="scan"/>
+    <xacro:hokuyo name="olei_lidar" xyz="0 0 1.515" rpy="0 0 0" parent="base_link" min_a="${-pi}" max_a="${pi}" topic="scan"/>
     <!-- VERTICAL 3D Olei Lidar  -->
     <!-- <xacro:velodyne16 name="olei_vertical" xyz="0.2 0 1" rpy="0 ${pi*1/4} 0" parent="base_link"/> -->
@@ -61,12 +81,12 @@
     <!-- depth_cam -->
     <xacro:include filename="$(find urdf_basic_shapes)/sensors/depth_cam.urdf.xacro"/>
-    <xacro:depth_cam name="cameraF" xyz=".2 0 ${.815-.075}" rpy="0 0 0" parent="base_link"/>
-    <!-- <xacro:depth_cam name="cameraF" xyz=".2 0 ${.76-.075}" rpy="0 0 0" parent="base_link"/> -->
-    <xacro:depth_cam name="cameraB" xyz="-.3 0 ${.6-.075}" rpy="0 0 ${pi}" parent="base_link"/>
-    <xacro:depth_cam name="cameraL" xyz="0 0.4 ${.9-.075}" rpy="${pi/2} 0 ${pi - 0.610865}" parent="base_link"/>
-    <xacro:depth_cam name="cameraR" xyz="0 -.4 ${.9-.075}" rpy="${-pi/2} 0 ${pi + 0.610865}" parent="base_link"/>
+    <xacro:depth_cam name="cameraF"      xyz=".230 0 ${.855-.075}" rpy="0 0 0" parent="base_link"/>
+    <xacro:depth_cam name="cameraF_down"    xyz=".140 0 ${.360-.075}" rpy="0 0 0" parent="base_link"/>
+    <xacro:depth_cam name="cameraB" xyz="-.3 0 ${.71-.075}" rpy="0 0 ${pi}" parent="base_link"/>
+    <xacro:depth_cam name="cameraL" xyz="0 ${0.71031/2} ${.4275-.075}" rpy="${pi/2} 0 ${pi - 0.610865}" parent="base_link"/>
+    <xacro:depth_cam name="cameraR" xyz="0 -${0.71031/2} ${.4275-.075}" rpy="${-pi/2} 0 ${pi + 0.610865}" parent="base_link"/>
     <!-- Sonar -->
     <xacro:include filename="$(find urdf_basic_shapes)/sensors/sonar.urdf.xacro"/>
-    <xacro:sonar name="sonarR" xyz="-1.1 -.05 .05" rpy="0 -.0872665 ${pi + 0.174533}" parent="base_link" min_a="-0.05" max_a="0.05" topic="sonarR"/>
-    <xacro:sonar name="sonarL" xyz="-1.1 0.05 .05" rpy="0 -.0872665 ${pi - 0.174533}" parent="base_link" min_a="-0.05" max_a="0.05" topic="sonarL"/>
+    <xacro:sonar name="sonarR" xyz="-${1.1-0.00331} -.05 .05" rpy="0 -.0872665 ${pi + 0.174533}" parent="base_link" min_a="-0.05" max_a="0.05" topic="sonarR"/>
+    <xacro:sonar name="sonarL" xyz="-${1.1-0.00331} .05 .05" rpy="0 -.0872665 ${pi - 0.174533}" parent="base_link" min_a="-0.05" max_a="0.05" topic="sonarL"/>
 </robot>

File: urdf/diff_wheel_control.urdf.xacro (robot description, xacro)
@@ -14,5 +14,5 @@
             <type>transmission_interface/SimpleTransmission</type>
             <joint name="left_wheel_joint">
-                <hardwareInterface>VelocityJointInterface</hardwareInterface>
+                <hardwareInterface>hardware_interface/VelocityJointInterface</hardwareInterface>
             </joint>
             <actuator name="left_wheel_actuator">
@@ -31,5 +31,5 @@
             <type>transmission_interface/SimpleTransmission</type>
             <joint name="right_wheel_joint">
-                <hardwareInterface>VelocityJointInterface</hardwareInterface>
+                <hardwareInterface>hardware_interface/VelocityJointInterface</hardwareInterface>
             </joint>
             <actuator name="right_wheel_actuator">

Commit message: update URDF file

File: examples/tko_robot.urdf.xacro (robot description, xacro)
@@ -27,15 +27,15 @@
     </joint>
     <!-- hands -->
-    <xacro:cube name="handR" x=".6365" y=".095" z=".100" ori="-${.6365/2}  0 0" rpy="0 0 0" rgb="Blue" m="10" friction="${standard_friction}"/>
+    <xacro:cube name="handR" x=".6365" y=".171" z=".175" ori="-${.6365/2}  0 ${.175/2}" rpy="0 0 0" rgb="Blue" m="10" friction="${standard_friction}"/>
     <joint name="handR_joint" type="fixed">
         <parent link="base_link"/>
         <child link="handR"/>
-        <origin xyz="-.2475 -.3775 0.585" rpy="0 0 0"/>
+        <origin xyz="-.2475 -.3775 0.575" rpy="0 0 0"/>
     </joint>
-    <xacro:cube name="handL" x=".6365" y=".095" z=".100" ori="-${.6365/2} 0 0" rpy="0 0 0" rgb="Blue" m="10" friction="${standard_friction}"/>
+    <xacro:cube name="handL" x=".6365" y=".171" z=".175" ori="-${.6365/2} 0 ${.175/2}" rpy="0 0 0" rgb="Blue" m="10" friction="${standard_friction}"/>
     <joint name="handL_joint" type="fixed">
         <parent link="base_link"/>
         <child link="handL"/>
-        <origin xyz="-.2475 .3775 0.585" rpy="0 0 0"/>
+        <origin xyz="-.2475 .3775 0.575" rpy="0 0 0"/>
     </joint>
     <!-- tail -->
@@ -66,7 +66,7 @@
     <!-- Hokuyo Laser Back-->
     <xacro:include filename="$(find urdf_basic_shapes)/sensors/hokuyo.urdf.xacro"/>
-    <xacro:hokuyo name="scan_back" xyz="-.9765 0 0" rpy="${pi} 0 ${pi}" parent="base_link" min_a="${-pi/2}" max_a="${pi/2}" topic="/lidarBack/scan"/>
+    <xacro:hokuyo name="scan_back" xyz="-.9765 0 0" rpy="${pi} 0 ${pi}" parent="base_link" min_a="${-pi/18}" max_a="${pi/18}" topic="/lidarBack/scan"/>
     <!-- Hokuyo Laser Front-->
-    <xacro:hokuyo name="scan_front" xyz=".14 0.0 .077" rpy="0 0 0" parent="base_link" min_a="${-pi/2}" max_a="${pi/2}" topic="/lidarFront/scan"/>
+    <xacro:hokuyo name="scan_front" xyz=".14 0.0 0.23" rpy="0 0 0" parent="base_link" min_a="${-pi/2}" max_a="${pi/2}" topic="/lidarFront/scan"/>
     <!-- TOP 3D Olei Lidar  -->
     <xacro:include filename="$(find urdf_basic_shapes)/sensors/velodyne.urdf.xacro"/>
@@ -81,9 +81,9 @@
     <!-- depth_cam -->
     <xacro:include filename="$(find urdf_basic_shapes)/sensors/depth_cam.urdf.xacro"/>
-    <xacro:depth_cam name="cameraF"      xyz=".230 0 ${.855-.075}" rpy="0 0 0" parent="base_link"/>
-    <xacro:depth_cam name="cameraF_down"    xyz=".140 0 ${.360-.075}" rpy="0 0 0" parent="base_link"/>
-    <xacro:depth_cam name="cameraB" xyz="-.3 0 ${.71-.075}" rpy="0 0 ${pi}" parent="base_link"/>
+    <xacro:depth_cam name="cameraF"      xyz=".230 0 ${.8540-.075}" rpy="0 0 0" parent="base_link"/>
+    <xacro:depth_cam name="cameraF_down" xyz=".140 0 ${.3625-.075}" rpy="0 0 0" parent="base_link"/>
     <xacro:depth_cam name="cameraL" xyz="0 ${0.71031/2} ${.4275-.075}" rpy="${pi/2} 0 ${pi - 0.610865}" parent="base_link"/>
     <xacro:depth_cam name="cameraR" xyz="0 -${0.71031/2} ${.4275-.075}" rpy="${-pi/2} 0 ${pi + 0.610865}" parent="base_link"/>
+    <xacro:depth_cam name="cameraB" xyz="-.3 0 ${.7045-.075}" rpy="0 0 ${pi}" parent="base_link"/>
     <!-- Sonar -->
     <xacro:include filename="$(find urdf_basic_shapes)/sensors/sonar.urdf.xacro"/>
