Commit message: TKOH_commit

File: examples/tko_robot_rise3D.urdf.xacro (robot description, xacro)
@@ -81,12 +81,12 @@
     <xacro:imu name="imu" xyz="0 0 0" rpy="0 0 0" parent="base_link"/>
     <!-- depth_cam -->
-    <xacro:include filename="$(find urdf_basic_shapes)/sensors/depth_cam.urdf.xacro"/>
+    <!-- <xacro:include filename="$(find urdf_basic_shapes)/sensors/depth_cam.urdf.xacro"/> -->
     <!-- <xacro:depth_cam name="cameraF"      xyz=".230 0 ${.8540-.075}" rpy="0 0 0" parent="base_link"/> -->
-    <link name="cameraF_link"/>
+    <!-- <link name="cameraF_link"/>
     <joint name="cameraF_joint" type="fixed">
         <parent link="base_link"/>
         <child link="cameraF_link"/>
         <origin xyz="0.230 0.0 ${.8540-.075}" rpy="0.0 0.0 0.0"/>
-    </joint>
+    </joint> -->
     <!-- <xacro:depth_cam name="cameraF_down" xyz=".140 -0.05 ${.3625-.075}" rpy="-${pi} 0 0" parent="base_link"/> -->
     <!-- <link name="cameraF_down"/> -->
@@ -97,17 +97,17 @@
     </joint> -->
     <!-- <xacro:depth_cam name="cameraL" xyz="0 ${0.71031/2} ${.4275-.075}" rpy="${pi/2} 0 ${pi - 0.610865}" parent="base_link"/> -->
-    <link name="cameraL_link"/>
+    <!-- <link name="cameraL_link"/>
     <joint name="cameraL_joint" type="fixed">
         <parent link="base_link"/>
         <child link="cameraL_link"/>
         <origin xyz="0 ${0.71031/2} ${.4275-.075}" rpy="${pi/2} 0 ${pi - 0.610865}"/>
-    </joint>
+    </joint> -->
     <!-- <xacro:depth_cam name="cameraR" xyz="0 -${0.71031/2} ${.4275-.075}" rpy="${-pi/2} 0 ${pi + 0.610865}" parent="base_link"/> -->
-    <link name="cameraR_link"/>
+    <!-- <link name="cameraR_link"/>
     <joint name="cameraR_joint" type="fixed">
         <parent link="base_link"/>
         <child link="cameraR_link"/>
         <origin xyz="0 -${0.71031/2} ${.4275-.075}" rpy="${-pi/2} 0 ${pi + 0.610865}"/>
-    </joint>
+    </joint> -->
     <!-- <xacro:depth_cam name="cameraB" xyz="-.3 0 ${.7045-.075}" rpy="0 0 ${pi}" parent="base_link"/> -->
     <!-- <link name="cameraB_link"/>
@@ -119,58 +119,8 @@
     <!-- usb_cam -->
     <xacro:include filename="$(find urdf_basic_shapes)/sensors/usb_cam.urdf.xacro" />
-    <xacro:usb_cam name="cameraF_down" xyz="0.140 -0.0 ${0.3625-0.075}" rpy="0.0 0.0 0.0" parent="base_link" rate="6" />
+    <!-- <xacro:usb_cam name="cameraF_down" xyz="0.140 -0.0 ${0.3625-0.075}" rpy="0.0 0.0 0.0" parent="base_link" rate="6" /> -->
+    <xacro:usb_cam name="cameraF_down" xyz="0.140 -0.03 ${0.3625-0.075}" rpy="0.0 0.0 0.0" parent="base_link" rate="6" />
     <xacro:usb_cam name="cameraB" xyz="-.3 0 ${.7045-.075}" rpy="0 0 ${pi}" parent="base_link" rate="6" />
     <!-- <xacro:usb_cam name="cameraT" xyz="-.08 0 1.59396" rpy="0 -${pi/2} 0" parent="base_link" rate="6" />     -->
-    <!-- TOF -->
-    <!-- Left TOF sensor -->
-    <!-- <link name="dep_cam_left_link"/> -->
-    <!-- <visual>
-        <geometry>
-            <box size="${tof_sensor_length} ${tof_sensor_width} ${tof_sensor_height}" />
-        </geometry>
-        <material name="yellow">
-            <color rgba="1 1 0 1" />
-        </material>
-    </visual>
-    <collision>
-        <geometry>
-            <box size="${tof_sensor_length} ${tof_sensor_width} ${tof_sensor_height}" />
-        </geometry>
-    </collision>
-    <inertial>
-        <mass value="0.1" />
-        <inertia ixx="0.000166" ixy="0" ixz="0" iyy="0.000166" iyz="0" izz="0.000166" />
-    </inertial>
-    </link> -->
-    <!-- <joint name="dep_cam_left_joint" type="fixed">
-        <parent link="base_link" />
-        <child link="dep_cam_left_link" />
-        <origin xyz="-0.10412 0.35523 0.41992" rpy="0.0 0.0 ${pi - 0.610865}" />
-    </joint> -->
-    <!-- Right TOF sensor -->
-    <!-- <link name="dep_cam_right_link"/> -->
-    <!-- <visual>
-        <geometry>
-            <box size="${tof_sensor_length} ${tof_sensor_width} ${tof_sensor_height}" />
-        </geometry>
-        <material name="yellow">
-            <color rgba="1 1 0 1" />
-        </material>
-    </visual>
-    <collision>
-        <geometry>
-            <box size="${tof_sensor_length} ${tof_sensor_width} ${tof_sensor_height}" />
-        </geometry>
-    </collision>
-    <inertial>
-        <mass value="0.1" />
-        <inertia ixx="0.000166" ixy="0" ixz="0" iyy="0.000166" iyz="0" izz="0.000166" />
-    </inertial>
-    </link> -->
-    <!-- <joint name="dep_cam_right_joint" type="fixed">
-        <parent link="base_link" />
-        <child link="dep_cam_right_link" />
-        <origin xyz="-0.10412 -0.35523 0.41992" rpy="0.0 0.0 ${pi + 0.610865}" />
-    </joint> -->
     <!-- Sonar -->
     <!-- <xacro:include filename="$(find urdf_basic_shapes)/sensors/sonar.urdf.xacro"/>
