Commit message: new deliverybot with two lidar

File: examples/deliverybot/deliverybot.urdf (robot description, URDF)
Before this commit: robot deliverybot, 16 links, 15 joints
Links:
- removed link back_scan
- removed link front_scan
- added link scan_back, mass 1e-5; collision box size=0.1 0.1 0.1; visual box size=0.1 0.1 0.1
- added link scan_front, mass 1e-5; collision box size=0.1 0.1 0.1; visual box size=0.1 0.1 0.1
Joints:
- removed joint back_scan_joint
- removed joint front_scan_joint
- added joint scan_back_joint: type fixed, parent base_link, child scan_back, origin xyz=-.25 0 .05 rpy=0 0 0, axis 0 1 0
- added joint scan_front_joint: type fixed, parent base_link, child scan_front, origin xyz=.25 0 .05 rpy=0 3.141592653589793 0, axis 0 1 0

File: examples/deliverybot/deliverybot.urdf.xacro (robot description, xacro)
@@ -52,6 +52,6 @@
     <!-- Hokuyo Laser -->
     <xacro:include filename="$(find urdf_basic_shapes)/sensors/hokuyo.urdf.xacro"/>
-    <xacro:hokuyo name="front_scan" xyz=".25 0 .05" rpy="0 ${pi} 0" parent="base_link" min_a="${-pi}" max_a="${pi}"/>
-    <xacro:hokuyo name="back_scan" xyz="-.25 0 .05" rpy="0 0 0" parent="base_link" min_a="${-pi}" max_a="${pi}"/>
+    <xacro:hokuyo name="scan_front" xyz=".25 0 .05" rpy="0 ${pi} 0" parent="base_link" min_a="${-pi}" max_a="${pi}"/>
+    <xacro:hokuyo name="scan_back" xyz="-.25 0 .05" rpy="0 0 0" parent="base_link" min_a="${-pi}" max_a="${pi}"/>
      <!-- imu -->
     <xacro:include filename="$(find urdf_basic_shapes)/sensors/imu.urdf.xacro"/>

Commit message: modify diff wheel to fix bug

File: examples/deliverybot/deliverybot.urdf (robot description, URDF)
Before this commit: robot deliverybot, 16 links, 15 joints
Links:
- link left_wheel: geometry collision sphere radius=0.1; visual cylinder length=0.05 radius=0.1
- link right_wheel: geometry collision sphere radius=0.1; visual cylinder length=0.05 radius=0.1

File: examples/deliverybot/deliverybot.urdf.xacro (robot description, xacro)
@@ -35,5 +35,5 @@
     <!-- the parent link should be the center of wheel axis -->
     <xacro:include filename="$(find urdf_basic_shapes)/urdf/diff_wheel.urdf.xacro"/>
-    <xacro:diff_wheel wheeldiam="0.2" h=".05" wheel_separation=".38" parent="base_link" friction="1000" rgb="Black" odom_topic="odom" pub_tf="false"/>
+    <xacro:diff_wheel wheeldiam="0.2" h=".05" wheel_separation=".38" parent="base_link" friction="${wheel_friction}" rgb="Black" odom_topic="odom" pub_tf="false"/>
     <!-- caster wheel back -->
     <xacro:ball name="casterwheel_back" r="0.1" ori="0 0 0" rpy="0 0 0" rgb="Grey" m=".1" friction="${sliding_friction}"/>

File: urdf/basic_shapes.gazebo.xacro (robot description, xacro)
@@ -5,5 +5,5 @@
   <xacro:property name="standard_friction" value="0.2" />
   <xacro:property name="wheel_friction" value="10000.0" />
-  <xacro:property name="sliding_friction" value="0.1" />
+  <xacro:property name="sliding_friction" value="0.001" />
     <xacro:macro name="gazebo_params" params="name rgb friction">
         <gazebo reference="${name}">

File: urdf/basic_shapes.urdf.xacro (robot description, xacro)
@@ -67,3 +67,22 @@
     <xacro:gazebo_params name="${name}" rgb="${rgb}" friction="${friction}"/>
   </xacro:macro>
+  <xacro:macro name="wheel" params="name r h ori rpy rgb m friction">
+    <link name="${name}">
+        <visual>
+          <origin xyz="${ori}" rpy="${rpy}"/>
+          <geometry>
+              <cylinder radius="${r}" length="${h}"/>
+          </geometry>
+          <material name="${rgb}"/>
+        </visual>
+        <collision>
+        <origin xyz="${ori}" rpy="${rpy}" />
+        <geometry>
+            <sphere radius="${r}" />   <!--use shpere here to reduce the point of contract to a infinit small point-->
+        </geometry>
+        </collision>
+        <xacro:solid_cylinder_inertia m="${m}" r="${r}" h="${h}"/>
+    </link>
+    <xacro:gazebo_params name="${name}" rgb="${rgb}" friction="${friction}"/>
+  </xacro:macro>
 </robot>

File: urdf/diff_wheel.urdf.xacro (robot description, xacro)
@@ -3,5 +3,5 @@
     <!-- differential drive macro -->
     <xacro:macro name="diff_wheel" params=" wheeldiam h wheel_separation parent friction rgb odom_topic:=odom pub_tf:=true">
-        <xacro:cylinder_shape name="left_wheel" r="${wheeldiam/2}" h="${h}" ori="0 0 0" rpy="0 0 0" rgb="${rgb}" m="0.1" friction="${friction}"/>
+        <xacro:wheel name="left_wheel" r="${wheeldiam/2}" h="${h}" ori="0 0 0" rpy="0 0 0" rgb="${rgb}" m="0.1" friction="${friction}"/>
         <joint name="left_wheel_joint" type="continuous">
             <axis xyz="0 0 1" rpy="0 0 0" />
@@ -10,5 +10,5 @@
             <origin xyz="0 ${wheel_separation/2} 0" rpy="${-pi/2} 0 0"/>
         </joint>
-        <xacro:cylinder_shape name="right_wheel" r="${wheeldiam/2}" h="${h}" ori="0 0 0" rpy="0 0 0" rgb="${rgb}" m="0.1" friction="${friction}"/>
+        <xacro:wheel name="right_wheel" r="${wheeldiam/2}" h="${h}" ori="0 0 0" rpy="0 0 0" rgb="${rgb}" m="0.1" friction="${friction}"/>
         <joint name="right_wheel_joint" type="continuous">
             <axis xyz="0 0 1" rpy="0 0 0" />
