Commit message: mod lidar

File: examples/deliverybot/deliverybot.urdf.xacro (robot description, xacro)
@@ -52,6 +52,6 @@
     <!-- Hokuyo Laser -->
     <xacro:include filename="$(find urdf_basic_shapes)/sensors/hokuyo.urdf.xacro"/>
-    <xacro:hokuyo name="scan_front" xyz=".25 0 .05" rpy="0 ${pi} 0" parent="base_link" min_a="${-pi}" max_a="${pi}"/>
-    <xacro:hokuyo name="scan_back" xyz="-.25 0 .05" rpy="0 0 0" parent="base_link" min_a="${-pi}" max_a="${pi}"/>
+    <xacro:hokuyo name="scan_front" xyz=".25 0 .05" rpy="0 ${pi} 0" parent="base_link" min_a="${-pi}" max_a="${pi}" topic="scan"/>
+    <xacro:hokuyo name="scan_back" xyz="-.25 0 .05" rpy="0 0 0" parent="base_link" min_a="${-pi}" max_a="${pi}" topic="scan_back"/>
      <!-- imu -->
     <xacro:include filename="$(find urdf_basic_shapes)/sensors/imu.urdf.xacro"/>

File: sensors/hokuyo.urdf.xacro (robot description, xacro)
@@ -1,5 +1,5 @@
 <?xml version="1.0"?>
 <robot name="hokuyo" xmlns:xacro="http://wiki.ros.org/xacro">
-    <xacro:macro name="hokuyo" params="name parent xyz rpy min_a max_a">
+    <xacro:macro name="hokuyo" params="name parent xyz rpy min_a max_a topic">
         <link name="${name}">
             <collision>
@@ -56,5 +56,5 @@
                 <plugin name="gazebo_ros_${name}_controller" filename="libgazebo_ros_ray_sensor.so">
                 <ros>
-                    <remapping>~/out:=${name}</remapping>
+                    <remapping>~/out:=${topic}</remapping>
                 </ros>
                 <output_type>sensor_msgs/LaserScan</output_type>

Commit message: add mesh for deliverybot

File: examples/deliverybot/deliverybot.urdf.xacro (robot description, xacro)
@@ -5,5 +5,24 @@
     <link name="base_footprint"/>
     <!--cylinder base_link -->
-    <xacro:cylinder_shape name="base_link" r="0.25" h="1.2" ori="0 0 .7" rpy="0 0 0" rgb="White" m="10" friction="${standard_friction}"/>
+    <!-- <xacro:cylinder_shape name="base_link" r="0.25" h="1.2" ori="0 0 .7" rpy="0 0 0" rgb="White" m="10" friction="${standard_friction}"/> -->
+    <link name="base_link">
+        <visual>
+            <origin xyz="0.0 0.0 0.0" rpy="0.0 0.0 ${-pi/2}"/>
+            <geometry>
+                <!-- <cylinder radius="0.25" length="1.2"/> -->
+                <mesh filename="file://$(find urdf_basic_shapes)/meshes/deliverybot.dae"/>
+            </geometry>
+            <material name="LightGrey">
+                <color rgba="0.7 0.7 0.7 1.0"/>
+            </material>
+        </visual>
+        <collision>
+            <origin xyz="0.0 0.0 0.7" rpy="0.0 0.0 0.0"/>
+            <geometry>
+                <cylinder radius="0.25" length="1.2"/>
+            </geometry>
+        </collision>
+        <xacro:solid_cylinder_inertia m="10" r=".25" h="1.2"/>
+    </link>
     <joint name="base_joint" type="fixed">
         <parent link="base_footprint"/>
@@ -12,12 +31,12 @@
     </joint>
     <!-- cubic screen -->
-    <xacro:cube name="screen" x=".15" y=".3" z=".4" ori=".25 0 1" rpy="0 0 0" rgb="Blue" m="1" friction="${standard_friction}"/>
+    <!-- <xacro:cube name="screen" x=".15" y=".3" z=".4" ori=".25 0 1" rpy="0 0 0" rgb="Blue" m="1" friction="${standard_friction}"/>
     <joint name="screen_joint" type="fixed">
         <parent link="base_link"/>
         <child link="screen"/>
         <origin xyz="0 0 0" rpy="0 0 0"/>
-    </joint>
+    </joint> -->
     <!-- cubic butt -->
-    <xacro:cube name="butt" x=".3" y=".5" z=".4" ori="0 0 0" rpy="0 0 0" rgb="White" m="1" friction="${standard_friction}"/>
+    <xacro:cube name="butt" x=".3" y=".4" z=".4" ori="0 0 0" rpy="0 0 0" rgb="White" m="10" friction="${standard_friction}"/>
     <joint name="butt_joint" type="fixed">
         <parent link="base_link"/>
@@ -26,10 +45,10 @@
     </joint>
     <!-- Head  -->
-    <xacro:ball name="head" r="0.25" ori="0 0 0" rpy="0 0 0" rgb="White" m="1" friction="${standard_friction}"/>
+    <!-- <xacro:ball name="head" r="0.25" ori="0 0 0" rpy="0 0 0" rgb="White" m="1" friction="${standard_friction}"/>
     <joint name="joint_head" type="fixed">
         <parent link="base_link"/>
         <child link="head"/>
         <origin xyz="0 0 1.3" rpy="0 0 0"/>
-    </joint>
+    </joint> -->
     <!-- diff drive -->
     <!-- the parent link should be the center of wheel axis -->
@@ -41,5 +60,5 @@
         <parent link="base_link"/>
         <child link="casterwheel_back"/>
-        <origin xyz="-.25 0 -.0" rpy="0 0 0"/>
+        <origin xyz="-.2 0 -.0" rpy="0 0 0"/>
     </joint>
     <!-- caster wheel front -->
@@ -48,17 +67,17 @@
         <parent link="base_link"/>
         <child link="casterwheel_front"/>
-        <origin xyz=".25 0 -.0" rpy="0 0 0"/>
+        <origin xyz=".2 0 -.0" rpy="0 0 0"/>
     </joint>
     <!-- Hokuyo Laser -->
     <xacro:include filename="$(find urdf_basic_shapes)/sensors/hokuyo.urdf.xacro"/>
     <xacro:hokuyo name="scan_front" xyz=".25 0 .05" rpy="0 ${pi} 0" parent="base_link" min_a="${-pi}" max_a="${pi}" topic="scan"/>
-    <xacro:hokuyo name="scan_back" xyz="-.25 0 .05" rpy="${pi} 0 0" parent="base_link" min_a="${-pi}" max_a="${pi}" topic="back/scan"/>
-     <!-- imu -->
+    <xacro:hokuyo name="scan_back" xyz="-.30 0 .05" rpy="${pi} 0 0" parent="base_link" min_a="${-pi}" max_a="${pi}" topic="back/scan"/>
+    <!-- depth_cam -->
+    <xacro:include filename="$(find urdf_basic_shapes)/sensors/depth_cam.urdf.xacro"/>
+    <xacro:depth_cam name="cameraL" xyz=".22 0.19 .3" rpy="0 0 ${pi/4}" parent="base_link"/>
+    <xacro:depth_cam name="cameraR" xyz=".22 -.19 .3" rpy="${pi} 0 -${pi/4}" parent="base_link"/>
+    <!-- imu -->
     <xacro:include filename="$(find urdf_basic_shapes)/sensors/imu.urdf.xacro"/>
     <xacro:imu name="imu" xyz="0 0 0" rpy="0 0 0" parent="cameraL"/>
     <!-- better not use "/" in "name" can cause some warnings -->
-    <!-- depth_cam -->
-    <xacro:include filename="$(find urdf_basic_shapes)/sensors/depth_cam.urdf.xacro"/>
-    <xacro:depth_cam name="cameraL" xyz=".19 0.18 .3" rpy="0 0 ${pi/4}" parent="base_link"/>
-    <xacro:depth_cam name="cameraR" xyz=".19 -.18 .3" rpy="${pi} 0 -${pi/4}" parent="base_link"/>
 </robot>

Commit message: match cam to reality

File: examples/deliverybot/deliverybot.urdf.xacro (robot description, xacro)
@@ -75,9 +75,9 @@
     <!-- depth_cam -->
     <xacro:include filename="$(find urdf_basic_shapes)/sensors/depth_cam.urdf.xacro"/>
-    <xacro:depth_cam name="cameraL" xyz=".22 0.19 .3" rpy="0 0 ${pi/4}" parent="base_link"/>
-    <xacro:depth_cam name="cameraR" xyz=".22 -.19 .3" rpy="${pi} 0 -${pi/4}" parent="base_link"/>
+    <xacro:depth_cam name="camL" xyz=".22 0.19 .3" rpy="0 0 ${pi/4}" parent="base_link"/>
+    <xacro:depth_cam name="camR" xyz=".22 -.19 .3" rpy="${pi} 0 -${pi/4}" parent="base_link"/>
     <!-- imu -->
     <xacro:include filename="$(find urdf_basic_shapes)/sensors/imu.urdf.xacro"/>
-    <xacro:imu name="imu" xyz="0 0 0" rpy="0 0 0" parent="cameraL"/>
+    <xacro:imu name="imu" xyz="0 0 0" rpy="0 0 0" parent="camL_link"/>
     <!-- better not use "/" in "name" can cause some warnings -->
 </robot>

File: sensors/depth_cam.urdf.xacro (robot description, xacro)
@@ -2,5 +2,5 @@
 <robot name="depth_cam" xmlns:xacro="http://wiki.ros.org/xacro">
     <xacro:macro name="depth_cam" params="name parent xyz rpy">
-    <link name="${name}">
+    <link name="${name}_link">
       <visual>
         <origin xyz="0 0 0" rpy="${pi/2} 0 ${pi/2}"/>
@@ -26,5 +26,5 @@
     <joint name="${name}_joint" type="fixed">
       <parent link="${parent}"/>
-      <child link="${name}"/>
+      <child link="${name}_link"/>
       <origin xyz="${xyz}" rpy="${rpy}"/>
     </joint>
@@ -32,5 +32,5 @@
     <joint name="${name}_depth_joint" type="fixed">
       <origin xyz="0 0 0" rpy="${-pi/2} 0 ${-pi/2}"/>
-      <parent link="${name}"/>
+      <parent link="${name}_link"/>
       <child link="${name}_depth_frame"/>
     </joint>

Commit message: mod for real robot

File: examples/deliverybot/deliverybot.urdf.xacro (robot description, xacro)
@@ -8,5 +8,5 @@
     <link name="base_link">
         <visual>
-            <origin xyz="0.0 0.0 0.0" rpy="0.0 0.0 ${-pi/2}"/>
+            <origin xyz="0.0 0.0 -0.10" rpy="0.0 0.0 ${-pi/2}"/>
             <geometry>
                 <!-- <cylinder radius="0.25" length="1.2"/> -->
@@ -75,6 +75,6 @@
     <!-- depth_cam -->
     <xacro:include filename="$(find urdf_basic_shapes)/sensors/depth_cam.urdf.xacro"/>
-    <xacro:depth_cam name="camL" xyz=".22 0.19 .3" rpy="0 0 ${pi/4}" parent="base_link"/>
-    <xacro:depth_cam name="camR" xyz=".22 -.19 .3" rpy="${pi} 0 -${pi/4}" parent="base_link"/>
+    <xacro:depth_cam name="camL" xyz=".22 0.19 .2" rpy="0 0 ${pi/4}" parent="base_link"/>
+    <xacro:depth_cam name="camR" xyz=".22 -.19 .2" rpy="${pi} 0 -${pi/4}" parent="base_link"/>
     <!-- imu -->
     <xacro:include filename="$(find urdf_basic_shapes)/sensors/imu.urdf.xacro"/>

File: sensors/depth_cam.urdf.xacro (robot description, xacro)
@@ -29,5 +29,5 @@
       <origin xyz="${xyz}" rpy="${rpy}"/>
     </joint>
-    <link name="${name}_depth_frame"/>
+    <!-- <link name="${name}_depth_frame"/>
     <joint name="${name}_depth_joint" type="fixed">
       <origin xyz="0 0 0" rpy="${-pi/2} 0 ${-pi/2}"/>
@@ -70,5 +70,5 @@
         </plugin>
       </sensor>
-    </gazebo>
+    </gazebo> -->
   </xacro:macro>
 </robot>

Commit message: add usb_cam optical frame

File: examples/deliverybot/deliverybot.urdf.xacro (robot description, xacro)
@@ -79,5 +79,5 @@
     <!-- usb_cam -->
     <xacro:include filename="$(find urdf_basic_shapes)/sensors/usb_cam.urdf.xacro"/>
-    <xacro:usb_cam name="camF" xyz=".28 0 .125" rpy="0 0 0" parent="base_link"/>
+    <xacro:usb_cam name="camF" xyz=".28 0 .125" rpy="0 0 0" parent="base_link" rate="6"/>
     <!-- imu -->
     <xacro:include filename="$(find urdf_basic_shapes)/sensors/imu.urdf.xacro"/>

File: sensors/usb_cam.urdf.xacro (robot description, xacro)
@@ -1,5 +1,5 @@
 <?xml version="1.0"?>
 <robot name="usb_cam" xmlns:xacro="http://wiki.ros.org/xacro">
-    <xacro:macro name="usb_cam" params="name parent xyz rpy">
+    <xacro:macro name="usb_cam" params="name parent xyz rpy rate:=24">
     <xacro:cube name="${name}" x="0.015" y="0.03" z="0.03" ori="-.007 0 0" rpy="0 0 0" rgb="Red" m="0.02" friction="${standard_friction}"/>
     <joint name="${name}_joint" type="fixed">
@@ -8,8 +8,14 @@
       <origin xyz="${xyz}" rpy="${rpy}"/>
     </joint>
+    <link name="${name}_optical_frame"/>
+    <joint name="${name}_optical_joint" type="fixed">
+      <parent link="${name}"/>
+      <child link="${name}_optical_frame"/>
+      <origin xyz="0.0 0.0 0.0" rpy="${-pi/2} 0.0 ${-pi/2}"/>
+    </joint>
     <gazebo reference="${name}">
       <sensor name="${name}" type="camera">
         <visualize>true</visualize>
-        <update_rate>6.0</update_rate>
+        <update_rate>${rate}</update_rate>
         <camera name="${name}">
           <horizontal_fov>1.3962634</horizontal_fov>
@@ -36,5 +42,5 @@
           <alwaysOn>true</alwaysOn>
           <updateRate>0.0</updateRate>
-          <frame_name>${name}</frame_name>
+          <frame_name>${name}_optical_frame</frame_name>
           <distortionK1>0</distortionK1>
           <distortionK2>0</distortionK2>
