Commit message: get back mesh for sensors

File: sensors/VLP-16.urdf.xacro (robot description, xacro)
@@ -16,10 +16,12 @@
       <visual>
         <geometry>
-          <cylinder radius="0.0516" length="0.0717"/>
+          <!-- <cylinder radius="0.0516" length="0.0717"/> -->
+          <mesh filename="package://velodyne_description/meshes/VLP16_base_1.dae" />
         </geometry>
       </visual>
       <visual>
         <geometry>
-          <cylinder radius="0.0516" length="0.0717"/>
+          <!-- <cylinder radius="0.0516" length="0.0717"/> -->
+          <mesh filename="package://velodyne_description/meshes/VLP16_base_2.dae" />
         </geometry>
       </visual>
@@ -45,5 +47,6 @@
         <origin xyz="0 0 -0.0377"/>
         <geometry>
-          <cylinder radius="0.0516" length="0.0717"/>
+          <!-- <cylinder radius="0.0516" length="0.0717"/> -->
+          <mesh filename="package://velodyne_description/meshes/VLP16_scan.dae" />
         </geometry>
       </visual>

File: sensors/hokuyo.urdf.xacro (robot description, xacro)
@@ -12,6 +12,6 @@
             <origin xyz="0 0 0" rpy="0 0 0"/>
             <geometry>
-                <box size="0.1 0.1 0.1"/>
-                <!-- <mesh filename="package://urdf_basic_shapes/meshes/hokuyo.dae"/> -->
+                <!-- <box size="0.1 0.1 0.1"/> -->
+                <mesh filename="package://urdf_basic_shapes/meshes/hokuyo.dae"/>
             </geometry>
             </visual>

Commit message: fix mesh issue with gazebo

File: sensors/VLP-16.urdf.xacro (robot description, xacro)
@@ -17,5 +17,5 @@
         <geometry>
           <!-- <cylinder radius="0.0516" length="0.0717"/> -->
-          <mesh filename="package://velodyne_description/meshes/VLP16_base_1.dae" />
+          <mesh filename="$(find velodyne_description)/meshes/VLP16_base_1.dae" />
         </geometry>
       </visual>
@@ -23,5 +23,5 @@
         <geometry>
           <!-- <cylinder radius="0.0516" length="0.0717"/> -->
-          <mesh filename="package://velodyne_description/meshes/VLP16_base_2.dae" />
+          <mesh filename="$(find velodyne_description)/meshes/VLP16_base_2.dae" />
         </geometry>
       </visual>
@@ -48,5 +48,5 @@
         <geometry>
           <!-- <cylinder radius="0.0516" length="0.0717"/> -->
-          <mesh filename="package://velodyne_description/meshes/VLP16_scan.dae" />
+          <mesh filename="$(find velodyne_description)/meshes/VLP16_scan.dae" />
         </geometry>
       </visual>

File: sensors/depth_cam.urdf.xacro (robot description, xacro)
@@ -7,5 +7,5 @@
         <geometry>
           <!-- <box size="0.015 0.130 0.022"/> -->
-          <mesh filename="package://urdf_basic_shapes/meshes/intel_d435.dae"/>
+          <mesh filename="$(find urdf_basic_shapes)/meshes/intel_d435.dae"/>
         </geometry>
       </visual>

File: sensors/hokuyo.urdf.xacro (robot description, xacro)
@@ -13,5 +13,5 @@
             <geometry>
                 <!-- <box size="0.1 0.1 0.1"/> -->
-                <mesh filename="package://urdf_basic_shapes/meshes/hokuyo.dae"/>
+                <mesh filename="$(find urdf_basic_shapes)/meshes/hokuyo.dae"/>
             </geometry>
             </visual>

File: urdf/diff_wheel.urdf.xacro (robot description, xacro)
@@ -37,7 +37,8 @@
             <!-- <odometry_source>world</odometry_source> -->
             <!-- output -->
+            <robot_base_frame>base_footprint</robot_base_frame>
             <publish_odom>true</publish_odom>
             <publish_odom_tf>${pub_tf}</publish_odom_tf>
-            <publish_wheel_tf>false</publish_wheel_tf>
+            <publish_wheel_tf>true</publish_wheel_tf>
             <!-- <publish_wheel_joint_state>true</publish_wheel_joint_state> -->
             <!-- <publish_tf>true</publish_tf> -->

Commit message: fix mesh issue

File: sensors/VLP-16.urdf.xacro (robot description, xacro)
@@ -17,5 +17,6 @@
         <geometry>
           <!-- <cylinder radius="0.0516" length="0.0717"/> -->
-          <mesh filename="$(find velodyne_description)/meshes/VLP16_base_1.dae" />
+          <mesh filename="file://$(find velodyne_description)/meshes/VLP16_base_1.dae" />
+          <!-- <mesh filename="$(find velodyne_description)/meshes/VLP16_base_1.dae" /> -->
         </geometry>
       </visual>
@@ -23,5 +24,6 @@
         <geometry>
           <!-- <cylinder radius="0.0516" length="0.0717"/> -->
-          <mesh filename="$(find velodyne_description)/meshes/VLP16_base_2.dae" />
+          <mesh filename="file://$(find velodyne_description)/meshes/VLP16_base_2.dae" />
+          <!-- <mesh filename="$(find velodyne_description)/meshes/VLP16_base_2.dae" /> -->
         </geometry>
       </visual>

File: sensors/depth_cam.urdf.xacro (robot description, xacro)
@@ -6,6 +6,8 @@
         <origin xyz="0 0 0" rpy="${pi/2} 0 ${pi/2}"/>
         <geometry>
-          <!-- <box size="0.015 0.130 0.022"/> -->
-          <mesh filename="$(find urdf_basic_shapes)/meshes/intel_d435.dae"/>
+          <mesh filename="file://$(find urdf_basic_shapes)/meshes/intel_d435.dae" />
+          <!-- <mesh filename="$(find urdf_basic_shapes)/meshes/intel_d435.dae"/> -->
+          <box size=" 0.130 0.015 0.022"/>
+          <!-- <mesh filename="package://urdf_basic_shapes/meshes/intel_d435.dae"/> -->
         </geometry>
       </visual>

File: sensors/hokuyo.urdf.xacro (robot description, xacro)
@@ -13,5 +13,6 @@
             <geometry>
                 <!-- <box size="0.1 0.1 0.1"/> -->
-                <mesh filename="$(find urdf_basic_shapes)/meshes/hokuyo.dae"/>
+                <mesh filename="file://$(find urdf_basic_shapes)/meshes/hokuyo.dae" />
+                <!-- <mesh filename="$(find urdf_basic_shapes)/meshes/hokuyo.dae"/> -->
             </geometry>
             </visual>
