Commit message: change output topic of info

File: sensors/depth_cam.urdf.xacro (robot description, xacro)
@@ -1,5 +1,6 @@
 <?xml version="1.0"?>
-<robot name="depth_cam" xmlns:xacro="http://wiki.ros.org/xacro">
-    <xacro:macro name="depth_cam" params="name parent xyz rpy">
+<robot name="depth_cam"
+  xmlns:xacro="http://wiki.ros.org/xacro">
+  <xacro:macro name="depth_cam" params="name parent xyz rpy">
     <xacro:property name="r200_cam_rgb_px" value="0.005"/>
     <xacro:property name="r200_cam_rgb_py" value="0.018"/>
@@ -14,7 +15,7 @@
     <link name="${name}_link">
       <visual>
-      <origin xyz="0 0 0" rpy="1.57 0 1.57"/>
+        <origin xyz="0 0 0" rpy="1.57 0 1.57"/>
         <geometry>
-        <mesh filename="package://urdf_basic_shapes/meshes/intel_d435.dae" />
+          <mesh filename="package://urdf_basic_shapes/meshes/intel_d435.dae" />
         </geometry>
       </visual>
@@ -26,71 +27,71 @@
       </collision>
     </link>
-  <joint name="${name}_rgb_joint" type="fixed">
-    <origin xyz="${r200_cam_rgb_px} ${r200_cam_rgb_py} ${r200_cam_rgb_pz}" rpy="0 0 0"/>
-    <parent link="${name}_link"/>
-    <child link="${name}_rgb_frame"/>
-  </joint>
-  <link name="${name}_rgb_frame"/>
-  <joint name="${name}_rgb_optical_joint" type="fixed">
-    <origin xyz="0 0 0" rpy="-1.57 0 -1.57"/>
-    <parent link="${name}_rgb_frame"/>
-    <child link="${name}_rgb_optical_frame"/>
-  </joint>
-  <link name="${name}_rgb_optical_frame"/>
-  <joint name="${name}_depth_joint" type="fixed">
-    <origin xyz="${r200_cam_rgb_px} ${r200_cam_rgb_py + r200_cam_depth_offset} ${r200_cam_rgb_pz}" rpy="0 0 0"/>
-    <parent link="${name}_link"/>
-    <child link="${name}_depth_frame"/>
-  </joint>
-  <link name="${name}_depth_frame"/>
-  <joint name="${name}_depth_optical_joint" type="fixed">
-    <origin xyz="0 0 0" rpy="-1.57 0 -1.57"/>
-    <parent link="${name}_depth_frame"/>
-    <child link="${name}_depth_optical_frame"/>
-  </joint>
-  <link name="${name}_depth_optical_frame"/>
-  <gazebo reference="${name}_rgb_frame">
-    <sensor type="depth" name="realsense_R200">
-      <always_on>true</always_on>
-      <visualize>$(arg camera_visual)</visualize>
-      <camera>
+    <joint name="${name}_rgb_joint" type="fixed">
+      <origin xyz="${r200_cam_rgb_px} ${r200_cam_rgb_py} ${r200_cam_rgb_pz}" rpy="0 0 0"/>
+      <parent link="${name}_link"/>
+      <child link="${name}_rgb_frame"/>
+    </joint>
+    <link name="${name}_rgb_frame"/>
+    <joint name="${name}_rgb_optical_joint" type="fixed">
+      <origin xyz="0 0 0" rpy="-1.57 0 -1.57"/>
+      <parent link="${name}_rgb_frame"/>
+      <child link="${name}_rgb_optical_frame"/>
+    </joint>
+    <link name="${name}_rgb_optical_frame"/>
+    <joint name="${name}_depth_joint" type="fixed">
+      <origin xyz="${r200_cam_rgb_px} ${r200_cam_rgb_py + r200_cam_depth_offset} ${r200_cam_rgb_pz}" rpy="0 0 0"/>
+      <parent link="${name}_link"/>
+      <child link="${name}_depth_frame"/>
+    </joint>
+    <link name="${name}_depth_frame"/>
+    <joint name="${name}_depth_optical_joint" type="fixed">
+      <origin xyz="0 0 0" rpy="-1.57 0 -1.57"/>
+      <parent link="${name}_depth_frame"/>
+      <child link="${name}_depth_optical_frame"/>
+    </joint>
+    <link name="${name}_depth_optical_frame"/>
+    <gazebo reference="${name}_rgb_frame">
+      <sensor type="depth" name="realsense_R200">
+        <always_on>true</always_on>
+        <visualize>$(arg camera_visual)</visualize>
+        <camera>
           <horizontal_fov>1.3439</horizontal_fov>
           <image>
-              <width>1920</width>
-              <height>1080</height>
-              <format>R8G8B8</format>
+            <width>1920</width>
+            <height>1080</height>
+            <format>R8G8B8</format>
           </image>
           <depth_camera></depth_camera>
           <clip>
-              <near>0.03</near>
-              <far>100</far>
+            <near>0.03</near>
+            <far>100</far>
           </clip>
-      </camera>
-      <plugin name="${name}_controller" filename="libgazebo_ros_openni_kinect.so">
-        <baseline>0.2</baseline>
-        <alwaysOn>true</alwaysOn>
-        <updateRate>30.0</updateRate>
-        <cameraName>${name}</cameraName>
-        <frameName>${name}_rgb_optical_frame</frameName>
-        <imageTopicName>rgb/image_raw</imageTopicName>
-        <depthImageTopicName>depth/image_raw</depthImageTopicName>
-        <pointCloudTopicName>depth/points</pointCloudTopicName>
-        <cameraInfoTopicName>rgb/${name}_info</cameraInfoTopicName>
-        <depthImageCameraInfoTopicName>depth/${name}_info</depthImageCameraInfoTopicName>
-        <pointCloudCutoff>0.4</pointCloudCutoff>
-            <hackBaseline>0.07</hackBaseline>
-            <distortionK1>0.0</distortionK1>
-            <distortionK2>0.0</distortionK2>
-            <distortionK3>0.0</distortionK3>
-            <distortionT1>0.0</distortionT1>
-            <distortionT2>0.0</distortionT2>
-        <CxPrime>0.0</CxPrime>
-        <Cx>0.0</Cx>
-        <Cy>0.0</Cy>
-        <focalLength>0</focalLength>
-        <hackBaseline>0</hackBaseline>
-      </plugin>
-    </sensor>
-  </gazebo>
+        </camera>
+        <plugin name="${name}_controller" filename="libgazebo_ros_openni_kinect.so">
+          <baseline>0.2</baseline>
+          <alwaysOn>true</alwaysOn>
+          <updateRate>30.0</updateRate>
+          <cameraName>${name}</cameraName>
+          <frameName>${name}_rgb_optical_frame</frameName>
+          <imageTopicName>rgb/image_raw</imageTopicName>
+          <depthImageTopicName>depth/image_raw</depthImageTopicName>
+          <pointCloudTopicName>depth/points</pointCloudTopicName>
+          <cameraInfoTopicName>rgb/camera_info</cameraInfoTopicName>
+          <depthImageCameraInfoTopicName>depth/camera_info</depthImageCameraInfoTopicName>
+          <pointCloudCutoff>0.4</pointCloudCutoff>
+          <hackBaseline>0.07</hackBaseline>
+          <distortionK1>0.0</distortionK1>
+          <distortionK2>0.0</distortionK2>
+          <distortionK3>0.0</distortionK3>
+          <distortionT1>0.0</distortionT1>
+          <distortionT2>0.0</distortionT2>
+          <CxPrime>0.0</CxPrime>
+          <Cx>0.0</Cx>
+          <Cy>0.0</Cy>
+          <focalLength>0</focalLength>
+          <hackBaseline>0</hackBaseline>
+        </plugin>
+      </sensor>
+    </gazebo>
   </xacro:macro>
 </robot>

Commit message: update cam topics

File: sensors/depth_cam.urdf.xacro (robot description, xacro)
@@ -1,5 +1,6 @@
 <?xml version="1.0"?>
-<robot name="depth_cam" xmlns:xacro="http://wiki.ros.org/xacro">
-    <xacro:macro name="depth_cam" params="name parent xyz rpy">
+<robot name="depth_cam"
+  xmlns:xacro="http://wiki.ros.org/xacro">
+  <xacro:macro name="depth_cam" params="name parent xyz rpy">
     <xacro:property name="r200_cam_rgb_px" value="0.005"/>
     <xacro:property name="r200_cam_rgb_py" value="0.018"/>
@@ -14,7 +15,7 @@
     <link name="${name}_link">
       <visual>
-      <origin xyz="0 0 0" rpy="1.57 0 1.57"/>
+        <origin xyz="0 0 0" rpy="1.57 0 1.57"/>
         <geometry>
-        <mesh filename="package://urdf_basic_shapes/meshes/intel_d435.dae" />
+          <mesh filename="package://urdf_basic_shapes/meshes/intel_d435.dae" />
         </geometry>
       </visual>
@@ -26,71 +27,71 @@
       </collision>
     </link>
-  <joint name="${name}_rgb_joint" type="fixed">
-    <origin xyz="${r200_cam_rgb_px} ${r200_cam_rgb_py} ${r200_cam_rgb_pz}" rpy="0 0 0"/>
-    <parent link="${name}_link"/>
-    <child link="${name}_rgb_frame"/>
-  </joint>
-  <link name="${name}_rgb_frame"/>
-  <joint name="${name}_rgb_optical_joint" type="fixed">
-    <origin xyz="0 0 0" rpy="-1.57 0 -1.57"/>
-    <parent link="${name}_rgb_frame"/>
-    <child link="${name}_rgb_optical_frame"/>
-  </joint>
-  <link name="${name}_rgb_optical_frame"/>
-  <joint name="${name}_depth_joint" type="fixed">
-    <origin xyz="${r200_cam_rgb_px} ${r200_cam_rgb_py + r200_cam_depth_offset} ${r200_cam_rgb_pz}" rpy="0 0 0"/>
-    <parent link="${name}_link"/>
-    <child link="${name}_depth_frame"/>
-  </joint>
-  <link name="${name}_depth_frame"/>
-  <joint name="${name}_depth_optical_joint" type="fixed">
-    <origin xyz="0 0 0" rpy="-1.57 0 -1.57"/>
-    <parent link="${name}_depth_frame"/>
-    <child link="${name}_depth_optical_frame"/>
-  </joint>
-  <link name="${name}_depth_optical_frame"/>
-  <gazebo reference="${name}_rgb_frame">
-    <sensor type="depth" name="realsense_R200">
-      <always_on>true</always_on>
-      <visualize>$(arg camera_visual)</visualize>
-      <camera>
+    <joint name="${name}_rgb_joint" type="fixed">
+      <origin xyz="${r200_cam_rgb_px} ${r200_cam_rgb_py} ${r200_cam_rgb_pz}" rpy="0 0 0"/>
+      <parent link="${name}_link"/>
+      <child link="${name}_rgb_frame"/>
+    </joint>
+    <link name="${name}_rgb_frame"/>
+    <joint name="${name}_rgb_optical_joint" type="fixed">
+      <origin xyz="0 0 0" rpy="-1.57 0 -1.57"/>
+      <parent link="${name}_rgb_frame"/>
+      <child link="${name}_rgb_optical_frame"/>
+    </joint>
+    <link name="${name}_rgb_optical_frame"/>
+    <joint name="${name}_depth_joint" type="fixed">
+      <origin xyz="${r200_cam_rgb_px} ${r200_cam_rgb_py + r200_cam_depth_offset} ${r200_cam_rgb_pz}" rpy="0 0 0"/>
+      <parent link="${name}_link"/>
+      <child link="${name}_depth_frame"/>
+    </joint>
+    <link name="${name}_depth_frame"/>
+    <joint name="${name}_depth_optical_joint" type="fixed">
+      <origin xyz="0 0 0" rpy="-1.57 0 -1.57"/>
+      <parent link="${name}_depth_frame"/>
+      <child link="${name}_depth_optical_frame"/>
+    </joint>
+    <link name="${name}_depth_optical_frame"/>
+    <gazebo reference="${name}_rgb_frame">
+      <sensor type="depth" name="realsense_R200">
+        <always_on>true</always_on>
+        <visualize>$(arg camera_visual)</visualize>
+        <camera>
           <horizontal_fov>1.3439</horizontal_fov>
           <image>
-              <width>1920</width>
-              <height>1080</height>
-              <format>R8G8B8</format>
+            <width>1920</width>
+            <height>1080</height>
+            <format>R8G8B8</format>
           </image>
           <depth_camera></depth_camera>
           <clip>
-              <near>0.03</near>
-              <far>100</far>
+            <near>0.03</near>
+            <far>100</far>
           </clip>
-      </camera>
-      <plugin name="${name}_controller" filename="libgazebo_ros_openni_kinect.so">
-        <baseline>0.2</baseline>
-        <alwaysOn>true</alwaysOn>
-        <updateRate>30.0</updateRate>
-        <cameraName>${name}</cameraName>
-        <frameName>${name}_rgb_optical_frame</frameName>
-        <imageTopicName>rgb/image_raw</imageTopicName>
-        <depthImageTopicName>depth/image_raw</depthImageTopicName>
-        <pointCloudTopicName>depth/points</pointCloudTopicName>
-        <cameraInfoTopicName>rgb/${name}_info</cameraInfoTopicName>
-        <depthImageCameraInfoTopicName>depth/${name}_info</depthImageCameraInfoTopicName>
-        <pointCloudCutoff>0.4</pointCloudCutoff>
-            <hackBaseline>0.07</hackBaseline>
-            <distortionK1>0.0</distortionK1>
-            <distortionK2>0.0</distortionK2>
-            <distortionK3>0.0</distortionK3>
-            <distortionT1>0.0</distortionT1>
-            <distortionT2>0.0</distortionT2>
-        <CxPrime>0.0</CxPrime>
-        <Cx>0.0</Cx>
-        <Cy>0.0</Cy>
-        <focalLength>0</focalLength>
-        <hackBaseline>0</hackBaseline>
-      </plugin>
-    </sensor>
-  </gazebo>
+        </camera>
+        <plugin name="${name}_controller" filename="libgazebo_ros_openni_kinect.so">
+          <baseline>0.2</baseline>
+          <alwaysOn>true</alwaysOn>
+          <updateRate>30.0</updateRate>
+          <cameraName>${name}</cameraName>
+          <frameName>${name}_depth_optical_frame</frameName>
+          <imageTopicName>rgb/image_raw</imageTopicName>
+          <depthImageTopicName>depth/image_raw</depthImageTopicName>
+          <pointCloudTopicName>depth/color/points</pointCloudTopicName>
+          <cameraInfoTopicName>rgb/${name}_info</cameraInfoTopicName>
+          <depthImageCameraInfoTopicName>depth/${name}_info</depthImageCameraInfoTopicName>
+          <pointCloudCutoff>0.4</pointCloudCutoff>
+          <hackBaseline>0.07</hackBaseline>
+          <distortionK1>0.0</distortionK1>
+          <distortionK2>0.0</distortionK2>
+          <distortionK3>0.0</distortionK3>
+          <distortionT1>0.0</distortionT1>
+          <distortionT2>0.0</distortionT2>
+          <CxPrime>0.0</CxPrime>
+          <Cx>0.0</Cx>
+          <Cy>0.0</Cy>
+          <focalLength>0</focalLength>
+          <hackBaseline>0</hackBaseline>
+        </plugin>
+      </sensor>
+    </gazebo>
   </xacro:macro>
 </robot>

Commit message: match cam with realsense

File: sensors/depth_cam.urdf.xacro (robot description, xacro)
@@ -3,7 +3,7 @@
   xmlns:xacro="http://wiki.ros.org/xacro">
   <xacro:macro name="depth_cam" params="name parent xyz rpy">
-    <xacro:property name="r200_cam_rgb_px" value="0.005"/>
-    <xacro:property name="r200_cam_rgb_py" value="0.018"/>
-    <xacro:property name="r200_cam_rgb_pz" value="0.013"/>
+    <xacro:property name="r200_cam_color_px" value="0.005"/>
+    <xacro:property name="r200_cam_color_py" value="0.018"/>
+    <xacro:property name="r200_cam_color_pz" value="0.013"/>
     <xacro:property name="r200_cam_depth_offset" value="0.01"/>
     <xacro:arg name="camera_visual" default="false"/>
@@ -27,18 +27,18 @@
       </collision>
     </link>
-    <joint name="${name}_rgb_joint" type="fixed">
-      <origin xyz="${r200_cam_rgb_px} ${r200_cam_rgb_py} ${r200_cam_rgb_pz}" rpy="0 0 0"/>
+    <joint name="${name}_color_joint" type="fixed">
+      <origin xyz="${r200_cam_color_px} ${r200_cam_color_py} ${r200_cam_color_pz}" rpy="0 0 0"/>
       <parent link="${name}_link"/>
-      <child link="${name}_rgb_frame"/>
+      <child link="${name}_color_frame"/>
     </joint>
-    <link name="${name}_rgb_frame"/>
-    <joint name="${name}_rgb_optical_joint" type="fixed">
+    <link name="${name}_color_frame"/>
+    <joint name="${name}_color_optical_joint" type="fixed">
       <origin xyz="0 0 0" rpy="-1.57 0 -1.57"/>
-      <parent link="${name}_rgb_frame"/>
-      <child link="${name}_rgb_optical_frame"/>
+      <parent link="${name}_color_frame"/>
+      <child link="${name}_color_optical_frame"/>
     </joint>
-    <link name="${name}_rgb_optical_frame"/>
+    <link name="${name}_color_optical_frame"/>
     <joint name="${name}_depth_joint" type="fixed">
-      <origin xyz="${r200_cam_rgb_px} ${r200_cam_rgb_py + r200_cam_depth_offset} ${r200_cam_rgb_pz}" rpy="0 0 0"/>
+      <origin xyz="${r200_cam_color_px} ${r200_cam_color_py + r200_cam_depth_offset} ${r200_cam_color_pz}" rpy="0 0 0"/>
       <parent link="${name}_link"/>
       <child link="${name}_depth_frame"/>
@@ -51,5 +51,5 @@
     </joint>
     <link name="${name}_depth_optical_frame"/>
-    <gazebo reference="${name}_rgb_frame">
+    <gazebo reference="${name}_color_frame">
       <sensor type="depth" name="realsense_R200">
         <always_on>true</always_on>
@@ -74,8 +74,8 @@
           <cameraName>${name}</cameraName>
           <frameName>${name}_depth_optical_frame</frameName>
-          <imageTopicName>rgb/image_raw</imageTopicName>
+          <imageTopicName>color/image_raw</imageTopicName>
           <depthImageTopicName>depth/image_raw</depthImageTopicName>
           <pointCloudTopicName>depth/color/points</pointCloudTopicName>
-          <cameraInfoTopicName>rgb/${name}_info</cameraInfoTopicName>
+          <cameraInfoTopicName>color/${name}_info</cameraInfoTopicName>
           <depthImageCameraInfoTopicName>depth/${name}_info</depthImageCameraInfoTopicName>
           <pointCloudCutoff>0.4</pointCloudCutoff>

Commit message: put back camera to gazebo

File: sensors/depth_cam.urdf.xacro (robot description, xacro)
@@ -29,5 +29,5 @@
       <origin xyz="${xyz}" rpy="${rpy}"/>
     </joint>
-    <!-- <link name="${name}_depth_frame"/>
+    <link name="${name}_depth_frame"/>
     <joint name="${name}_depth_joint" type="fixed">
       <origin xyz="0 0 0" rpy="${-pi/2} 0 ${-pi/2}"/>
@@ -35,6 +35,6 @@
       <child link="${name}_depth_frame"/>
     </joint>
-    <gazebo reference="${name}">
-      <sensor name="depth_${name}" type="depth">
+    <gazebo reference="${name}_link">
+      <sensor name="${name}" type="depth">
         <visualize>true</visualize>
         <update_rate>10.0</update_rate>
@@ -56,4 +56,11 @@
           <updateRate>0.0</updateRate>
           <frame_name>${name}_depth_frame</frame_name>
+          <ros>
+            <!-- <remapping>${name}/image_raw:=color/image_raw</remapping>
+            <remapping>${name}/depth/image_raw:=depth/image_rect_raw</remapping>
+            <remapping>${name}/camera_info:=camera_info</remapping>
+            <remapping>${name}/depth/camera_info:=depth/camera_info</remapping> -->
+            <remapping>${name}/points:=${name}/depth/color/points</remapping>
+          </ros>
           <pointCloudCutoff>0.5</pointCloudCutoff>
           <pointCloudCutoffMax>3.0</pointCloudCutoffMax>
@@ -70,5 +77,5 @@
         </plugin>
       </sensor>
-    </gazebo> -->
+    </gazebo>
   </xacro:macro>
 </robot>
