Commit message: fix imu

File: sensors/imu.urdf.xacro (robot description, xacro)
@@ -2,78 +2,31 @@
 <robot name="imu" xmlns:xacro="http://wiki.ros.org/xacro">
     <xacro:macro name="imu" params="name parent xyz rpy">
-        <link name="${name}"/>
+        <link name="${name}" />
         <joint name="${name}_joint" type="fixed">
             <axis xyz="0 0 0" />
-            <origin xyz="${xyz}" rpy="${rpy}"/>
-            <parent link="${parent}"/>
-            <child link="${name}"/>
+            <origin xyz="${xyz}" rpy="${rpy}" />
+            <parent link="${parent}" />
+            <child link="${name}" />
         </joint>
         <!-- imu -->
         <gazebo reference="${name}">
+            <gravity>true</gravity>
             <sensor name="${name}" type="imu">
-            <plugin filename="libgazebo_ros_imu_sensor.so" name="imu_plugin">
-                <ros>
-                <namespace></namespace>
-                <remapping>~/out:=${name}</remapping>
-                </ros>
-                <initial_orientation_as_reference>false</initial_orientation_as_reference>
-            </plugin>
-            <always_on>true</always_on>
-            <update_rate>200</update_rate>
-            <visualize>true</visualize>
-            <imu>
-                <angular_velocity>
-                <x>
-                    <noise type="gaussian">
-                    <mean>0.0</mean>
-                    <stddev>2e-4</stddev>
-                    <bias_mean>0.0000075</bias_mean>
-                    <bias_stddev>0.0000008</bias_stddev>
-                    </noise>
-                </x>
-                <y>
-                    <noise type="gaussian">
-                    <mean>0.0</mean>
-                    <stddev>2e-4</stddev>
-                    <bias_mean>0.0000075</bias_mean>
-                    <bias_stddev>0.0000008</bias_stddev>
-                    </noise>
-                </y>
-                <z>
-                    <noise type="gaussian">
-                    <mean>0.0</mean>
-                    <stddev>2e-4</stddev>
-                    <bias_mean>0.0000075</bias_mean>
-                    <bias_stddev>0.0000008</bias_stddev>
-                    </noise>
-                </z>
-                </angular_velocity>
-                <linear_acceleration>
-                <x>
-                    <noise type="gaussian">
-                    <mean>0.0</mean>
-                    <stddev>1.7e-2</stddev>
-                    <bias_mean>0.1</bias_mean>
-                    <bias_stddev>0.001</bias_stddev>
-                    </noise>
-                </x>
-                <y>
-                    <noise type="gaussian">
-                    <mean>0.0</mean>
-                    <stddev>1.7e-2</stddev>
-                    <bias_mean>0.1</bias_mean>
-                    <bias_stddev>0.001</bias_stddev>
-                    </noise>
-                </y>
-                <z>
-                    <noise type="gaussian">
-                    <mean>0.0</mean>
-                    <stddev>1.7e-2</stddev>
-                    <bias_mean>0.1</bias_mean>
-                    <bias_stddev>0.001</bias_stddev>
-                    </noise>
-                </z>
-                </linear_acceleration>
-            </imu>
+                <always_on>true</always_on>
+                <update_rate>200</update_rate>
+                <visualize>true</visualize>
+                <topic>${name}</topic>
+                <plugin filename="libgazebo_ros_imu_sensor.so" name="imu_plugin">
+                    <topicName>${name}</topicName>
+                    <remapping>~/out:=${name}</remapping>
+                    <bodyName>${name}</bodyName>
+                    <updateRateHZ>10.0</updateRateHZ>
+                    <gaussianNoise>0.0</gaussianNoise>
+                    <xyzOffset>0 0 0</xyzOffset>
+                    <rpyOffset>0 0 0</rpyOffset>
+                    <frame_name>${name}</frame_name>
+                    <initialOrientationAsReference>false</initialOrientationAsReference>
+                </plugin>
+                <pose>0 0 0 0 0 0</pose>
             </sensor>
         </gazebo>
