Commit message: hokuyo update frame id

File: sensors/hokuyo.urdf.xacro (robot description, xacro)
@@ -1,5 +1,5 @@
 <?xml version="1.0"?>
 <robot name="hokuyo" xmlns:xacro="http://wiki.ros.org/xacro">
-    <xacro:macro name="hokuyo" params="name parent xyz rpy topic frame_id">
+    <xacro:macro name="hokuyo" params="name parent xyz rpy topic">
         <link name="${name}">
             <collision>
@@ -31,5 +31,5 @@
             <sensor type="gpu_ray" name="head_hokuyo_sensor">
             <pose>0 0 0 0 0 0</pose>
-            <visualize>true</visualize>
+            <visualize>false</visualize>
             <update_rate>40</update_rate>
             <ray>
@@ -59,5 +59,5 @@
             <plugin name="gazebo_ros_head_hokuyo_controller" filename="libgazebo_ros_gpu_laser.so">
                 <topicName>${topic}</topicName>
-                <frameName>${frame_id}</frameName>
+                <frameName>${name}</frameName>
             </plugin>
             </sensor>

Commit message: geive default min max angle for lidar

File: sensors/hokuyo.urdf.xacro (robot description, xacro)
@@ -2,5 +2,5 @@
 <robot name="hokuyo"
     xmlns:xacro="http://wiki.ros.org/xacro">
-    <xacro:macro name="hokuyo" params="name parent xyz rpy min_a max_a topic=scan">
+    <xacro:macro name="hokuyo" params="name parent xyz rpy min_a=${-pi} max_a=${pi} topic=scan">
         <link name="${name}">
             <collision>
